File: CMDB_pcb_rev1/CM5IO.kicad_sch (KiCad schematic)
At the start: 7 parts, among them J1 POWER TERMINAL, J11 USB_C_Receptacle_USB2.0

Commit message: Update page descriptions, add MD describing post fabrication fixes
Other:
- company: Copyright © 2024 Raspberry Pi Ltd. -> AGH Drone Engineering
- title: Compute Module 5 IO Board - Top Level -> Compute Module Drone Board
Changed lines of the file:
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@@
 	(paper "A4")
 	(title_block
-		(title "Compute Module 5 IO Board - Top Level")
+		(title "Compute Module Drone Board")
+		(date "01.2026")
 		(rev "1")
-		(company "Copyright © 2024 Raspberry Pi Ltd.")
-		(comment 1 "www.raspberrypi.com")
+		(company "AGH Drone Engineering")
+		(comment 1 "Author: Piotr Kądziela")
 	)
 	(text "Connectors\n-------\nSDCARD\n40way RPI\nJumpers\nFan"
