File: CMDB_pcb_rev1/CM5_GPIO.kicad_sch (KiCad schematic)
At the start: 19 parts, among them J14 JST_SHBM04B-SRSS-TB, J2 Conn_02x06_Odd_Even, J7 Micro_SD_Card_Det, J8 THD-20-R, SW1 Right angle Tact button, U18 RT9742GGJ5

Commit message: Update page descriptions, add MD describing post fabrication fixes
Other:
- company: Copyright © 2024 Raspberry Pi Ltd. -> AGH Drone Engineering
- title: Compute Module 5 IO Board - GPIO - Ethernet -> Compute Module Drone Board
Changed lines of the file:
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@@
 	(paper "A4")
 	(title_block
-		(title "Compute Module 5 IO Board - GPIO - Ethernet")
+		(title "Compute Module Drone Board")
+		(date "01.2026")
 		(rev "1")
-		(company "Copyright © 2024 Raspberry Pi Ltd.")
-		(comment 1 "www.raspberrypi.com")
+		(company "AGH Drone Engineering")
+		(comment 1 "Author: Piotr Kądziela")
 	)
 	(text "40Way GPIO Header"
