File: CMDB_pcb_rev1/CM5_HighSpeed.kicad_sch (KiCad schematic)
At the start: 20 parts, among them J12 USB3_A, J16 Conn_01x22_Female, J22 46765-1301, J3 62674-161121ALF, J5 Conn_01x22_Female, U12 RT9742SNGV, U6 AP22653W6

Commit message: Update page descriptions, add MD describing post fabrication fixes
Other:
- company: Copyright © 2024 Raspberry Pi Ltd. -> AGH Drone Engineering
- title: Compute Module 5 IO Board - CM5 - Highspeed -> Compute Module Drone Board
Changed lines of the file:
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@@
 	(paper "A4")
 	(title_block
-		(title "Compute Module 5 IO Board - CM5 - Highspeed")
+		(title "Compute Module Drone Board")
+		(date "01.2026")
 		(rev "1")
-		(company "Copyright © 2024 Raspberry Pi Ltd.")
-		(comment 1 "www.raspberrypi.com")
+		(company "AGH Drone Engineering")
+		(comment 1 "Author: Piotr Kądziela")
 	)
 	(text "USB 3 Pairs P/N swapped to help routing"
