File: CMDB_pcb_rev1/psu.kicad_sch (KiCad schematic)
At the start: 20 parts, among them J4 J_PSU_EN

Commit message: Update page descriptions, add MD describing post fabrication fixes
Other:
- company: (none) -> AGH Drone Engineering
- title: (none) -> Compute Module Drone Board
Changed lines of the file:
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@@
 	(generator_version "9.0")
 	(paper "A4")
+	(title_block
+		(title "Compute Module Drone Board")
+		(date "01.2026")
+		(rev "1")
+		(company "AGH Drone Engineering")
+		(comment 1 "Author: Piotr Kądziela")
+	)
 	(junction
 		(at 134.62 101.6)
