File: pcb_CMDB_Adv/ethernet.kicad_sch (KiCad schematic)
At the start: 24 parts, among them IC1 KSZ8795CLXCC, J10 ETH1, J18 ETH2, J3 THD-02-R, Q1 AO3401A, U2 TPD4EUSB30, U3 MagJack-A70-112-331N126

Commit message: CMDB-Adv PCB WIP
Parts:
- removed C18, C23, C24, C25: 100n, Capacitor_SMD:C_0805_2012Metric_Pad1.18x1.45mm_HandSolder, symbol Device:C_Small
- removed C4: 100n, Capacitor_SMD:C_0805_2012Metric_Pad1.18x1.45mm_HandSolder, symbol Device:C
- removed D12: ETH4_Y, symbol Device:LED_Small_Filled
- removed D17: ETH4_G, symbol Device:LED_Small_Filled
- removed J10: ETH1, symbol CMDB_Adv:ARJM11-009
- removed J18: ETH2, symbol CMDB_Adv:ARJM11-009
- removed J3: THD-02-R, Connector_PinHeader_2.54mm:PinHeader_2x02_P2.54mm_Vertical, symbol Connector_Generic:Conn_02x02_Odd_Even
- removed Q1: AO3401A, Package_TO_SOT_SMD:SOT-23, symbol Transistor_FET:AO3401A
- removed R27, R33, R35, R36, R37, R38: 220R, symbol Device:R_Small
- removed U2: TPD4EUSB30, Package_SON:USON-10_2.5x1.0mm_P0.5mm, symbol CM5IO:TPD4EUSB30
- removed U3: MagJack-A70-112-331N126, CM5IO:TRJG0926HENL, symbol CM5IO:MagJack-A70-112-331N126
- added C26: 10uF, Capacitor_SMD:C_1206_3216Metric_Pad1.33x1.80mm_HandSolder, symbol Device:C_Small
- added C27, C28, C29, C32, C33, C34, C36, C37, C38, C40: 100nF, Capacitor_SMD:C_0402_2012Metric_Pad1.18x1.45mm_HandSolder, symbol Device:C_Small
- added C30, C31, C35, C39: 22uF, Capacitor_SMD:C_1206_3216Metric_Pad1.33x1.80mm_HandSolder, symbol Device:C
- added D11: BAT54A, Package_TO_SOT_SMD:SOT-23, symbol Diode:BAT54A
- added FB1, FB2, FB3, FB4: BLM21PG221SN1D, Inductor_SMD:L_0805_2012Metric_Pad1.05x1.20mm_HandSolder, symbol Device:FerriteBead_Small
- added R40: 10K, symbol Device:R_Small
- added R41: 1K, symbol Device:R_Small
- IC1: Height 1.6 -> (none); Manufacturer (none) -> Microchip; Manufacturer_Name Microchip -> (none); Manufacturer_Part_Number KSZ8795CLXCC -> (none); Mouser Part Number 998-KSZ8795CLXCC -> (none); Mouser Price/Stock https://www.mouser.co.uk/ProductDetail/Microchip-Technology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 -> (none); Part No. (none) -> KSZ8795CLXCC
- R39: value 220R -> 1K
Connections:
- net 3V3: now also D11.1, R40.2; no longer IC1.1 (VDD12A), IC1.12 (VDDAT33_2), IC1.2 (VDDAT33_1), IC1.34 (VDDIO_1), IC1.48 (VDDIO_2), IC1.70 (VDDIO_3), IC1.76 (VDDAT33_3)
- net GND: now also C26.2, C27.1, C28.1, C29.1, C30.1, C31.1, C32.1, C33.1, C34.1, C35.1, C36.1, C37.1, C38.1, C39.1, C40.1
- net LED3_1: now also R39.2; no longer R34.2
- net ETH2.TX_P: now reaches IC1.10 (TXP2)
- net ETH2.TX_N: now reaches IC1.11 (TXM2)
- net ETH3.RX_P: now reaches IC1.13 (RXP3)
- net ETH3.RX_N: now reaches IC1.14 (RXM3)
- net ETH3.TX_P: now reaches IC1.15 (TXP3)
- net ETH3.TX_N: now reaches IC1.16 (TXM3)
- net ETH4.RX_P: now reaches IC1.17 (RXP4)
- net ETH4.RX_N: now reaches IC1.18 (RXM4)
- net ETH4.TX_P: now reaches IC1.19 (TXP4)
- net ETH4.TX_N: now reaches IC1.20 (TXM4)
- net ETH1.RX_P: now reaches IC1.4 (RXP1)
- net ETH1.RX_N: now reaches IC1.5 (RXM1)
- net ETH1.TX_P: now reaches IC1.6 (TXP1)
- net ETH1.TX_N: now reaches IC1.7 (TXM1)
- net RST_N: now reaches IC1.72 (RST_N)
- net RST_N: now also C26.1, D11.3, R40.1
- net ETH2.RX_P: now reaches IC1.8 (RXP2)
- net ETH2.RX_N: now reaches IC1.9 (RXM2)
- net 1V2 renamed +VDD12D
- net +VDD12D: now also C35.2, C36.2, C37.2, C38.2, FB3.2; no longer IC1.73 (VDD12D_3)
- net LED1_0 renamed ETH1.LED_G
- net LED1_1 renamed ETH1.LED_Y
- net LED2_0 renamed ETH2.LED_G
- net LED2_1 renamed ETH2.LED_Y
- net LED3_G_LOW renamed LED3_0
- net LED3_0: now also R41.2
- net LED3_Y_HIGH renamed ETH3.LED_Y
- net ETH3.LED_Y: now also R34.2
- net LED4_0 renamed ETH4.LED_G
- net LED4_1 renamed ETH4.LED_Y
- new net +1V2: FB3.1, FB4.1
- new net +3V3: FB1.1, FB2.1
- new net +VDD12A: C39.2, C40.2, FB4.2, IC1.1 (VDD12A), IC1.73 (VDD12D_3)
- new net +VDDAT: C27.2, C28.2, C29.2, C30.2, FB1.2, IC1.12 (VDDAT33_2), IC1.2 (VDDAT33_1), IC1.76 (VDDAT33_3)
- new net +VDDIO: C31.2, C32.2, C33.2, C34.2, FB2.2, IC1.34 (VDDIO_1), IC1.48 (VDDIO_2), IC1.70 (VDDIO_3)
- new net ESP32_EN: D11.2
- new net ETH3.LED_G: R41.1
- no-connect marks 4 -> 2
Other:
- note added: "KSZ8795 is bootstraped by LED pullups/pulldowns. LED3_1 needs to be pulled down to enable RMII. Current limiting resistor is necessary."
- note added: "KSZ8795 reset sequencing Holds RST_N low ~100 ms after ESP32 boot"
- note added: "TODO: - zreviewować pod kątem zgodności z CMDB-Lite (LSHM) - Diody ethernet - TVS - ETH-GbE - Crystal"
- note removed: "Ethernet"
- note removed: "Ethernet POE Protection"
- note removed: "POE Header"
- note removed: "TODO - ETHERNET - remove connector, replace with small MOLEX"
- moved on the sheet: IC1, R28, R31

Commit message: CMDB_Adv WIP
Parts:
- removed C26: 10uF, Capacitor_SMD:C_1206_3216Metric_Pad1.33x1.80mm_HandSolder, symbol Device:C_Small
- removed D11: BAT54A, Package_TO_SOT_SMD:SOT-23, symbol Diode:BAT54A
- removed R40: 10K, symbol Device:R_Small
- added C42: 100nF, Capacitor_SMD:C_0402_1005Metric_Pad0.74x0.62mm_HandSolder, symbol Device:C_Small
- added FB5: BLM21PG221SN1D, Inductor_SMD:L_0805_2012Metric_Pad1.05x1.20mm_HandSolder, symbol Device:FerriteBead_Small
- added J1: RFShield_OnePiece, symbol Device:RFShield_OnePiece
- added R38: 4K7, Resistor_SMD:R_0805_2012Metric_Pad1.20x1.40mm_HandSolder, symbol Device:R_Small
- added Y1: ASE-25.000MHZ-LC-T, Oscillator:Oscillator_SMD_Abracon_ASE-4Pin_3.2x2.5mm, symbol Oscillator:ASE-xxxMHz
- C27, C28, C29, C32, C33, C34, C36, C37, C38, C40: footprint Capacitor_SMD:C_0402_2012Metric_Pad1.18x1.45mm_HandSolder -> Capacitor_SMD:C_0402_1005Metric_Pad0.74x0.62mm_HandSolder
- IC1: footprint QFP40P1200X1200X160-80N -> CMDB_Adv:QFP40P1200X1200X160-80N
- R28, R34, R39, R41: footprint (none) -> Resistor_SMD:R_0805_2012Metric_Pad1.20x1.40mm_HandSolder
- R33: renamed from R31; value 1K -> 330R; footprint (none) -> Resistor_SMD:R_0805_2012Metric_Pad1.20x1.40mm_HandSolder
Connections:
- net RST_N is gone; now on net SWITCH_RST_N: IC1.72 (RST_N)
- net +VDD12A: no longer IC1.73 (VDD12D_3)
- net +VDD12D: now also IC1.73 (VDD12D_3)
- net +VDDAT: now also FB5.1
- net +VDDIO: now also R38.1
- net GND: now also C42.1, J1.1 (Shield), Y1.2 (GND)
- net SWITCH_INT: now reaches IC1.23 (INTR_N)
- net SWITCH_INT: now also R38.2
- net RMII.TX_EN: now reaches IC1.29 (TXEN5/TXDS5_CTL)
- net RMII.TXD0: now reaches IC1.30 (TXD5_0)
- net RMII.TXD1: now reaches IC1.32 (TXD5_1)
- net RMII.REFCLK: now reaches IC1.44 (RXC5/GRXC5)
- net RMII.RXD0: now reaches IC1.45 (RXD5_0)
- net RMII.RXD1: now reaches IC1.46 (RXD5_1)
- net RMII.CRS_DV: now reaches IC1.51 (RXDV5/CRSDV5/RXD5_CTL)
- net at IC1.79 (XI): now also Y1.3 (OUT)
- net LED3_0: no longer names the net of IC1.25 (LED3_0), R41.2
- net LED3_1: no longer names the net of IC1.24 (LED3_1), R39.2
- new net +VDDOSC: C42.2, FB5.2, Y1.1 (EN), Y1.4 (Vdd)
- no-connect marks 2 -> 23
Other:
- note added: "Replace beads with 0R if they cause problems"
- note added: "Switch, ferrites and decoupling caps should be under this shield"
- note removed: "KSZ8795 reset sequencing Holds RST_N low ~100 ms after ESP32 boot"
- note removed: "TODO: - zreviewować pod kątem zgodności z CMDB-Lite (LSHM) - Diody ethernet - TVS - ETH-GbE - Crystal"
- moved on the sheet: IC1, R28, R33, R34, R39, R41

Commit message: WIP
Parts:
- removed J1: RFShield_OnePiece, symbol Device:RFShield_OnePiece
Other:
- note removed: "Switch, ferrites and decoupling caps should be under this shield"
Changed lines of the file:
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@@
 		)
 	)
-	(text "Switch, ferrites and \ndecoupling caps should \nbe under this shield"
-		(exclude_from_sim no)
-		(at 107.188 150.622 0)
-		(effects
-			(font
-				(size 1.27 1.27)
-			)
-		)
-	)
 	(text "Replace beads with 0R if\nthey cause problems"
 		(exclude_from_sim no)
@@
 	)
 	(symbol
-		(lib_id "power:GND")
-		(at 106.68 163.83 0)
-		(unit 1)
-		(body_style 1)
-		(exclude_from_sim no)
-		(in_bom yes)
-		(on_board yes)
-		(in_pos_files yes)
-		(dnp no)
-		(fields_autoplaced yes)
-		(property "Reference" "#PWR038"
-			(at 106.68 170.18 0)
-			(hide yes)
-			(show_name no)
-			(do_not_autoplace no)
-			(effects
-				(font
-					(size 1.27 1.27)
-				)
-			)
-		)
-		(property "Value" "GND"
-			(at 106.68 168.91 0)
-			(show_name no)
-			(do_not_autoplace no)
-			(effects
-				(font
-					(size 1.27 1.27)
-				)
-			)
-		)
-		(property "Footprint" ""
-			(at 106.68 163.83 0)
-			(hide yes)
-			(show_name no)
-			(do_not_autoplace no)
-			(effects
-				(font
-					(size 1.27 1.27)
-				)
-			)
-		)
-		(property "Datasheet" ""
-			(at 106.68 163.83 0)
-			(hide yes)
-			(show_name no)
-			(do_not_autoplace no)
-			(effects
-				(font
-					(size 1.27 1.27)
-				)
-			)
-		)
-		(property "Description" "Power symbol creates a global label with name \"GND\" , ground"
-			(at 106.68 163.83 0)
-			(hide yes)
-			(show_name no)
-			(do_not_autoplace no)
-			(effects
-				(font
-					(size 1.27 1.27)
-				)
-			)
-		)
-		(pin "1"
-		)
-		(instances
-			(project "CMDB_Adv"
-				(path "/e63e39d7-6ac0-4ffd-8aa3-1841a4541b55/7113be25-0166-4101-9dfa-c42ffe60d6fd"
-					(reference "#PWR038")
-					(unit 1)
-				)
-			)
-		)
-	)
-	(symbol
 		(lib_id "Device:R_Small")
 		(at 247.65 97.79 0)
@@
 					(unit 1)
 				)
-			)
-		)
-	)
-	(symbol
-		(lib_id "Device:RFShield_OnePiece")
-		(at 106.68 153.67 0)
-		(unit 1)
-		(body_style 1)
-		(exclude_from_sim no)
-		(in_bom yes)
-		(on_board yes)
-		(in_pos_files yes)
-		(dnp no)
-		(fields_autoplaced yes)
-		(property "Reference" "J1"
-			(at 123.19 152.3999 0)
-			(show_name no)
-			(do_not_autoplace no)
-			(effects
-				(font
-					(size 1.27 1.27)
-				)
-				(justify left)
-			)
-		)
-		(property "Value" "RFShield_OnePiece"
-			(at 123.19 154.9399 0)
-			(show_name no)
-			(do_not_autoplace no)
-			(effects
-				(font
-					(size 1.27 1.27)
-				)
-				(justify left)
-			)
-		)
-		(property "Footprint" ""
-			(at 106.68 156.21 0)
-			(hide yes)
-			(show_name no)
-			(do_not_autoplace no)
-			(effects
-				(font
-					(size 1.27 1.27)
-				)
-			)
-		)
-		(property "Datasheet" ""
-			(at 106.68 156.21 0)
-			(hide yes)
-			(show_name no)
-			(do_not_autoplace no)
-			(effects
-				(font
-					(size 1.27 1.27)
-				)
-			)
-		)
-		(property "Description" "One-piece EMI RF shielding cabinet"
-			(at 106.68 153.67 0)
-			(hide yes)
-			(show_name no)
-			(do_not_autoplace no)
-			(effects
-				(font
-					(size 1.27 1.27)
-				)
-			)
-		)
-		(pin "1"
-		)
-		(instances
-			(project "CMDB_Adv"
-				(path "/e63e39d7-6ac0-4ffd-8aa3-1841a4541b55/7113be25-0166-4101-9dfa-c42ffe60d6fd"
-					(reference "J1")
-					(unit 1)
-				)
