File: pcb_CMDB_Adv/CM5.kicad_sch (KiCad schematic)
At the start: 19 parts, among them J5 CONN_FAN, SW1 BT_PWR, SW2 SW_CONFIG, SW5 SW_WL_BT

Commit message: CMDB-Adv PCB WIP
Parts:
- removed SW5: SW_WL_BT, symbol Switch:SW_DIP_x02
- added J19: CONN_RTC, Connector_JST:JST_SH_BM02B-SRSS-TB_1x02-1MP_P1.00mm_Vertical, symbol Connector_Generic:Conn_01x02
- added JP11: GPIO9_SEL, Jumper:SolderJumper-3_P1.3mm_Open_RoundedPad1.0x1.5mm, symbol Jumper:SolderJumper_3_Open
- added JP3: ETH_Y_SEL, Jumper:SolderJumper-3_P1.3mm_Open_RoundedPad1.0x1.5mm, symbol Jumper:SolderJumper_3_Open
- added JP4: ETH_G_SEL, Jumper:SolderJumper-3_P1.3mm_Open_RoundedPad1.0x1.5mm, symbol Jumper:SolderJumper_3_Open
- added JP5: GPIO8_SEL, Jumper:SolderJumper-3_P1.3mm_Open_RoundedPad1.0x1.5mm, symbol Jumper:SolderJumper_3_Open
- D4, D6: Distributor Mouser -> (none); Part Description Green 572nm LED Indication - Discrete 2.2V 2-SMD, No Lead -> (none)
- D5: Distributor Mouser -> (none); Part Description Red 620nm LED Indication - Discrete 2.2V 2-SMD, No Lead -> (none)
- D7: Distributor Mouser -> (none)
- J5: Distributor TME -> (none); Part Description 4 pin vertical 1mm pitch connector -> (none)
- Module1: Distributor Mouser -> (none); Part Description 100 Position Connector Receptacle, Center Strip Contacts Su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 -> (none)
- R10, R7, R8, R9: Part Description Resistor 1K M1005 1% 63mW -> (none)
- R11: Part Description Resistor 10K M1005 1% 63mW -> (none)
- SW1: Distributor TME -> (none)
- SW2: Distributor TME -> (none); Part Description 8-pin micro dip-switch -> (none)
- TP6: value TP +3V3 RPi -> +3V3 RPi; Distributor nf -> (none); Part Description Test point -> (none)
- TP7, TP8: Distributor nf -> (none); Part Description Test point -> (none)
Connections:
- net +3.3v_STDB is gone; now on net GND: SW2.8
- net +3.3v_RPi: no longer Module1.78 (GPIO_VREF(1.8v/3.3v_Input)), Module1.84 (+3.3v_(Output)), Module1.86 (+3.3v_(Output)), TP6.1
- net +5v: no longer Module1.77 (+5v_(Input)), Module1.79 (+5v_(Input)), Module1.81 (+5v_(Input)), Module1.83 (+5v_(Input)), Module1.85 (+5v_(Input)), Module1.87 (+5v_(Input))
- net BT_nDis: now also SW2.9
- net GND: now also J19.1 (Pin_1); no longer JP2.2 (C), Module1.11 (Ethernet_Pair2_P), Module1.35 (ID_SC), Module1.4 (Ethernet_Pair1_P), Module1.41 (GPIO25), Module1.6 (Ethernet_Pair1_N), Module1.62 (SD_CMD)
- net GP.8: now also JP5.3 (B); no longer Module1.39 (GPIO8)
- net GP.9: now also JP11.3 (B); no longer Module1.40 (GPIO9)
- net PMIC_ENABLE: no longer SW2.12
- net SYNC_OUT: no longer SW2.14
- net WL_nDis: now also SW2.10
- net nACT_LED: now also TP7.1; no longer R10.2, R9.2
- net nPWR_LED: now also TP8.1
- net RPI_ETH_G: now reaches Module1.15 (Ethernet_nLED3(3.3v))
- net RPI_ETH_G: now also JP4.1 (A)
- net RPI_ETH_Y: now reaches Module1.17 (Ethernet_nLED2(3.3v))
- net RPI_ETH_Y: now also JP3.1 (A)
- net SD.DAT5: now reaches Module1.64 (SD_DAT5)
- net SD.DAT4: now reaches Module1.68 (SD_DAT4)
- net SD.DAT7: now reaches Module1.70 (SD_DAT7)
- net SD.DAT6: now reaches Module1.72 (SD_DAT6)
- net ETH0.P0_N renamed ETH.P0_N
- net ETH0.P0_P renamed ETH.P0_P
- net ETH0.P2_N renamed ETH.P2_N
- net ETH0.P3_N renamed ETH.P3_N
- net ETH0.P3_P renamed ETH.P3_P
- net VBAT renamed +3V3STB
- net +3V3STB: now also J19.2 (Pin_2); no longer SW2.9
- new net +3V3RPi: Module1.78 (GPIO_VREF(1.8v/3.3v_Input)), Module1.84 (+3.3v_(Output)), Module1.86 (+3.3v_(Output)), TP6.1
- new net +5V: Module1.77 (+5v_(Input)), Module1.79 (+5v_(Input)), Module1.81 (+5v_(Input)), Module1.83 (+5v_(Input)), Module1.85 (+5v_(Input)), Module1.87 (+5v_(Input))
- new net ETH.P1_N: Module1.6 (Ethernet_Pair1_N)
- new net ETH.P1_P: Module1.4 (Ethernet_Pair1_P)
- new net ETH.P2_P: Module1.11 (Ethernet_Pair2_P)
- new net ETH_LED_G: JP4.2 (C), R9.2
- new net ETH_LED_Y: JP3.2 (C), R10.2
- new net GP.25: Module1.41 (GPIO25)
- new net GPIO1_RAW: JP2.2 (C), Module1.35 (ID_SC)
- new net GPIO8_RAW: JP5.2 (C), Module1.39 (GPIO8)
- new net GPIO9_RAW: JP11.2 (C), Module1.40 (GPIO9)
- new net LED_G: JP4.3 (B)
- new net LED_Y: JP3.3 (B)
- new net PMIC_DISABLE: SW2.12
- new net SD.CMD: Module1.62 (SD_CMD)
- new net UART_PCTL_RX: JP11.1 (A)
- new net UART_PCTL_TX: JP5.1 (A)
- no-connect marks 9 -> 3
Other:
- note added: "TODO: DIP Size"
- note removed: "Force RPIBOOT = Jumper Pins 1-2"
- note removed: "TODO: - DIPy zamiast zwor?"
- moved on the sheet: D4, D5, D6, D7, J5, JP1, JP2, Module1A, R10, R11, R7, R8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

Commit message: CMDB_Adv WIP
Parts:
- Module1: Part No. 2x DF40C-100DS-0.4V(51) -> 2x DF40C-100DS-0.4V(51) / 10164227-1001A1RLF / 10164227-100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
Connections:
- net +3.3v is gone; now on net +3V3RPi: R11.1
- net +3.3v_RPi is gone; now on net +3V3RPi: D4.2 (A), D5.2 (A), D6.2 (A), D7.2 (A)
- net +5v is gone; now on net +5V: J5.1 (Pin_1)
- net PMIC_DISABLE is gone; now on net PMIC_ENABLE: SW2.12
- net nACT_LED: now also TP8.1; no longer TP7.1
- net nPWR_LED: now also TP7.1; no longer TP8.1
- net LED_G renamed ETH.LED_G
- net LED_Y renamed ETH.LED_Y
- net SYNC_OUT: no longer names the net of Module1.18 (Ethernet_SYNC_OUT(3.3v))
- no-connect marks 3 -> 4
Other:
- note added: "Short PMIC_ENABLE to disable RPi PMIC"
- moved on the sheet: JP3, JP4
Changed lines of the file:
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@@
 		(comment 1 "Author: Piotr Kądziela")
 	)
+	(text "Short PMIC_ENABLE \nto disable RPi PMIC\n"
+		(exclude_from_sim no)
+		(at 149.606 195.834 0)
+		(effects
+			(font
+				(size 1.27 1.27)
+			)
+			(justify left)
+		)
+	)
 	(text "RPi ETH ACT"
 		(exclude_from_sim no)
@@
 	)
 	(no_connect
+		(at 77.47 43.18)
+	)
+	(no_connect
 		(at 77.47 134.62)
 	)
@@
 	(wire
 		(pts
-			(xy 38.1 153.67) (xy 44.45 153.67)
+			(xy 34.29 153.67) (xy 44.45 153.67)
 		)
 		(stroke
@@
 	(wire
 		(pts
-			(xy 16.51 142.24) (xy 27.94 142.24)
+			(xy 12.7 142.24) (xy 24.13 142.24)
 		)
 		(stroke
@@
 	(wire
 		(pts
-			(xy 38.1 142.24) (xy 44.45 142.24)
+			(xy 34.29 142.24) (xy 44.45 142.24)
 		)
 		(stroke
@@
 	(wire
 		(pts
-			(xy 161.29 177.8) (xy 173.99 177.8)
-		)
-		(stroke
-			(width 0)
-			(type solid)
-		)
-	)
-	(wire
-		(pts
 			(xy 33.02 123.19) (xy 33.02 121.92)
 		)
@@
 	(wire
 		(pts
-			(xy 109.22 163.83) (xy 115.57 163.83)
+			(xy 106.68 163.83) (xy 115.57 163.83)
 		)
 		(stroke
@@
 	(wire
 		(pts
-			(xy 16.51 153.67) (xy 27.94 153.67)
+			(xy 12.7 153.67) (xy 24.13 153.67)
 		)
 		(stroke
@@
 	(wire
 		(pts
-			(xy 20.32 158.75) (xy 33.02 158.75)
+			(xy 16.51 158.75) (xy 29.21 158.75)
 		)
 		(stroke
@@
 	(wire
 		(pts
-			(xy 63.5 43.18) (xy 77.47 43.18)
-		)
-		(stroke
-			(width 0)
-			(type solid)
-		)
-	)
-	(wire
-		(pts
 			(xy 29.21 53.34) (xy 44.45 53.34)
 		)
@@
 	(wire
 		(pts
-			(xy 33.02 158.75) (xy 33.02 157.48)
+			(xy 29.21 158.75) (xy 29.21 157.48)
 		)
 		(stroke
@@
 	(wire
 		(pts
-			(xy 33.02 147.32) (xy 33.02 146.05)
+			(xy 29.21 147.32) (xy 29.21 146.05)
 		)
 		(stroke
@@
 	(wire
 		(pts
-			(xy 20.32 147.32) (xy 33.02 147.32)
+			(xy 16.51 147.32) (xy 29.21 147.32)
 		)
 		(stroke
@@
 		)
 	)
-	(label "+3.3v_RPi"
-		(at 53.34 165.1 180)
-		(effects
-			(font
-				(size 1.27 1.27)
-			)
-			(justify right bottom)
-		)
-	)
 	(label "GPIO8_RAW"
 		(at 20.32 123.19 0)
@@
 		)
 	)
-	(label "ETH0{GbETH}"
+	(label "ETH{GbETH}"
 		(at 34.29 158.75 0)
 		(effects
@@
 		)
 	)
-	(label "+3.3v"
-		(at 109.22 163.83 0)
-		(effects
-			(font
-				(size 1.27 1.27)
-			)
-			(justify left bottom)
-		)
-	)
 	(label "GPIO0_RAW"
 		(at 64.77 66.04 0)
@@
 		)
 	)
-	(label "nPWR_LED"
-		(at 82.55 186.69 180)
-		(effects
-			(font
-				(size 1.27 1.27)
-			)
-			(justify right bottom)
-		)
-	)
 	(label "nACT_LED"
 		(at 17.78 167.64 0)
@@
 		)
 	)
-	(label "LED_G"
+	(label "ETH.LED_G"
 		(at 44.45 153.67 180)
 		(effects
@@
 		)
 	)
-	(label "SYNC_OUT"
-		(at 63.5 43.18 0)
-		(effects
-			(font
-				(size 1.27 1.27)
-			)
-			(justify left bottom)
-		)
-	)
 	(label "HDMI1.CK_P"
 		(at 175.26 101.6 0)
@@
 	)
 	(label "RPI_ETH_G"
-		(at 16.51 153.67 0)
+		(at 12.7 153.67 0)
 		(effects
 			(font
@@
 		)
 	)
-	(label "nACT_LED"
-		(at 82.55 180.34 180)
-		(effects
-			(font
-				(size 1.27 1.27)
-			)
-			(justify right bottom)
-		)
-	)
 	(label "GP.24"
 		(at 151.13 78.74 180)
@@
 		)
 	)
-	(label "PMIC_DISABLE"
+	(label "PMIC_ENABLE"
 		(at 173.99 182.88 180)
 		(effects
@@
 		)
 	)
-	(label "+5v"
+	(label "+5V"
 		(at 104.14 171.45 0)
 		(effects
@@
 		)
 	)
+	(label "nPWR_LED"
+		(at 82.55 180.34 180)
+		(effects
+			(font
+				(size 1.27 1.27)
+			)
+			(justify right bottom)
+		)
+	)
 	(label "USB0.RX_N"
 		(at 175.26 55.88 0)
@@
 	)
 	(label "RPI_ETH_Y"
-		(at 16.51 142.24 0)
+		(at 12.7 142.24 0)
 		(effects
 			(font
@@
 		)
 	)
+	(label "nACT_LED"
+		(at 82.55 186.69 180)
+		(effects
+			(font
+				(size 1.27 1.27)
+			)
+			(justify right bottom)
+		)
+	)
 	(label "GP.20"
 		(at 151.13 55.88 180)
@@
 		)
 	)
-	(label "LED_Y"
+	(label "ETH.LED_Y"
 		(at 44.45 142.24 180)
 		(effects
@@
 	)
 	(label "ETH_LED_G"
-		(at 20.32 158.75 0)
+		(at 16.51 158.75 0)
 		(effects
 			(font
@@
 	)
 	(label "ETH_LED_Y"
-		(at 20.32 147.32 0)
+		(at 16.51 147.32 0)
 		(effects
 			(font
@@
 		)
 	)
+	(label "+3V3RPi"
+		(at 106.68 163.83 0)
+		(effects
+			(font
+				(size 1.27 1.27)
+			)
+			(justify left bottom)
+		)
+	)
 	(label "WL_nDis"
 		(at 153.67 134.62 180)
@@
 		)
 	)
+	(label "+3V3RPi"
+		(at 53.34 165.1 180)
+		(effects
+			(font
+				(size 1.27 1.27)
+			)
+			(justify right bottom)
+		)
+	)
 	(label "+5V"
 		(at 151.13 119.38 180)
@@
 	(symbol
 		(lib_id "Jumper:SolderJumper_3_Open")
-		(at 33.02 153.67 0)
+		(at 29.21 153.67 0)
 		(unit 1)
 		(body_style 1)
@@
 		(dnp no)
 		(property "Reference" "JP4"
-			(at 33.147 151.511 0)
+			(at 29.337 151.511 0)
 			(show_name no)
 			(do_not_autoplace no)
@@
 		)
 		(property "Value" "ETH_G_SEL"
-			(at 33.147 149.479 0)
+			(at 29.337 149.479 0)
 			(show_name no)
 			(do_not_autoplace no)
@@
 		)
 		(property "Footprint" "Jumper:SolderJumper-3_P1.3mm_Open_RoundedPad1.0x1.5mm"
-			(at 33.02 153.67 0)
+			(at 29.21 153.67 0)
 			(hide yes)
 			(show_name no)
@@
 		)
 		(property "Datasheet" ""
-			(at 33.02 153.67 0)
+			(at 29.21 153.67 0)
 			(hide yes)
 			(show_name no)
@@
 		)
 		(property "Description" "Solder Jumper, 3-pole, open"
-			(at 33.02 153.67 0)
+			(at 29.21 153.67 0)
 			(hide yes)
 			(show_name no)
@@
 			)
 		)
-		(property "Part No." "2x   DF40C-100DS-0.4V(51)"
+		(property "Part No." "2x   DF40C-100DS-0.4V(51) / 10164227-1001A1RLF  / 10164227-1004A1RLF / "
 			(at 110.49 78.74 0)
 			(hide yes)
@@
 	(symbol
 		(lib_id "Jumper:SolderJumper_3_Open")
-		(at 33.02 142.24 0)
+		(at 29.21 142.24 0)
 		(unit 1)
 		(body_style 1)
@@
 		(dnp no)
 		(property "Reference" "JP3"
-			(at 33.02 139.954 0)
+			(at 29.21 139.954 0)
 			(show_name no)
 			(do_not_autoplace no)
@@
 		)
 		(property "Value" "ETH_Y_SEL"
-			(at 31.75 138.176 0)
+			(at 27.94 138.176 0)
 			(show_name no)
 			(do_not_autoplace no)
@@
 		)
 		(property "Footprint" "Jumper:SolderJumper-3_P1.3mm_Open_RoundedPad1.0x1.5mm"
-			(at 33.02 142.24 0)
+			(at 29.21 142.24 0)
 			(hide yes)
 			(show_name no)
@@
 		)
 		(property "Datasheet" ""
-			(at 33.02 142.24 0)
+			(at 29.21 142.24 0)
 			(hide yes)
 			(show_name no)
@@
 		)
 		(property "Description" "Solder Jumper, 3-pole, open"
-			(at 33.02 142.24 0)
+			(at 29.21 142.24 0)
 			(hide yes)
 			(show_name no)
@@
 			)
 		)
-		(property "Part No." "2x   DF40C-100DS-0.4V(51)"
+		(property "Part No." "2x   DF40C-100DS-0.4V(51) / 10164227-1001A1RLF  / 10164227-1004A1RLF / "
 			(at 80.01 83.82 0)
 			(hide yes)

Commit message: WIP
Parts:
- added J26: Conn_01x03, symbol Connector_Generic:Conn_01x03
Connections:
- net BT_nDis: now also SW2.11; no longer SW2.9
- net PMIC_ENABLE: now also SW2.13; no longer SW2.12
- net PWR_BUT: no longer SW2.11
- net USBOTG: now also SW2.14; no longer SW2.13
- net WL_nDis: now also SW2.12; no longer SW2.10
Changed lines of the file:
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@@
 	(wire
 		(pts
-			(xy 173.99 187.96) (xy 161.29 187.96)
-		)
-		(stroke
-			(width 0)
-			(type default)
-		)
-	)
-	(wire
-		(pts
 			(xy 12.7 142.24) (xy 24.13 142.24)
 		)
@@
 	(wire
 		(pts
+			(xy 161.29 180.34) (xy 173.99 180.34)
+		)
+		(stroke
+			(width 0)
+			(type solid)
+		)
+	)
+	(wire
+		(pts
 			(xy 138.43 119.38) (xy 151.13 119.38)
 		)
@@
 	(wire
 		(pts
-			(xy 161.29 185.42) (xy 173.99 185.42)
-		)
-		(stroke
-			(width 0)
-			(type default)
-		)
-	)
-	(wire
-		(pts
 			(xy 43.18 182.88) (xy 43.18 190.5)
 		)
@@
 	(wire
 		(pts
-			(xy 161.29 182.88) (xy 173.99 182.88)
-		)
-		(stroke
-			(width 0)
-			(type solid)
-		)
-	)
-	(wire
-		(pts
 			(xy 69.85 186.69) (xy 82.55 186.69)
 		)
@@
 	(wire
 		(pts
+			(xy 173.99 182.88) (xy 161.29 182.88)
+		)
+		(stroke
+			(width 0)
+			(type default)
+		)
+	)
+	(wire
+		(pts
 			(xy 12.7 118.11) (xy 27.94 118.11)
 		)
@@
 		)
 	)
-	(wire
-		(pts
-			(xy 161.29 180.34) (xy 173.99 180.34)
-		)
-		(stroke
-			(width 0)
-			(type default)
-		)
-	)
 	(bus
 		(pts
@@
 	(wire
 		(pts
+			(xy 161.29 177.8) (xy 173.99 177.8)
+		)
+		(stroke
+			(width 0)
+			(type default)
+		)
+	)
+	(wire
+		(pts
 			(xy 138.43 25.4) (xy 151.13 25.4)
 		)
@@
 	(wire
 		(pts
+			(xy 173.99 185.42) (xy 161.29 185.42)
+		)
+		(stroke
+			(width 0)
+			(type default)
+		)
+	)
+	(wire
+		(pts
 			(xy 138.43 91.44) (xy 151.13 91.44)
 		)
@@
 	(wire
 		(pts
-			(xy 173.99 190.5) (xy 161.29 190.5)
-		)
-		(stroke
-			(width 0)
-			(type default)
-		)
-	)
-	(wire
-		(pts
 			(xy 115.57 163.83) (xy 115.57 165.1)
 		)
@@
 		)
 	)
-	(label "nACT_LED"
-		(at 17.78 167.64 0)
+	(label "PMIC_ENABLE"
+		(at 173.99 180.34 180)
 		(effects
 			(font
 				(size 1.27 1.27)
 			)
-			(justify left bottom)
+			(justify right bottom)
 		)
 	)
-	(label "WL_nDis"
-		(at 173.99 187.96 180)
+	(label "nACT_LED"
+		(at 17.78 167.64 0)
 		(effects
 			(font
 				(size 1.27 1.27)
 			)
-			(justify right bottom)
+			(justify left bottom)
 		)
 	)
@@
 		)
 	)
-	(label "PWR_BUT"
-		(at 173.99 185.42 180)
-		(effects
-			(font
-				(size 1.27 1.27)
-			)
-			(justify right bottom)
-		)
-	)
 	(label "ETH.LED_G"
 		(at 44.45 153.67 180)
@@
 		)
 	)
-	(label "BT_nDis"
-		(at 173.99 190.5 180)
+	(label "nACT_LED"
+		(at 153.67 48.26 180)
 		(effects
 			(font
@@
 		)
 	)
-	(label "nACT_LED"
-		(at 153.67 48.26 180)
+	(label "ETH.P1_P"
+		(at 64.77 25.4 0)
 		(effects
 			(font
 				(size 1.27 1.27)
 			)
-			(justify right bottom)
+			(justify left bottom)
 		)
 	)
-	(label "ETH.P1_P"
-		(at 64.77 25.4 0)
+	(label "USBOTG"
+		(at 173.99 177.8 180)
 		(effects
 			(font
 				(size 1.27 1.27)
 			)
-			(justify left bottom)
+			(justify right bottom)
 		)
 	)
@@
 		)
 	)
-	(label "PMIC_ENABLE"
-		(at 173.99 182.88 180)
-		(effects
-			(font
-				(size 1.27 1.27)
-			)
-			(justify right bottom)
-		)
-	)
 	(label "PCIe.nCLKREQ"
 		(at 175.26 22.86 0)
@@
 		)
 	)
-	(label "USBOTG"
-		(at 173.99 180.34 180)
-		(effects
-			(font
-				(size 1.27 1.27)
-			)
-			(justify right bottom)
-		)
-	)
 	(label "USBC.D_P"
 		(at 267.97 27.94 180)
@@
 		)
 	)
+	(label "WL_nDis"
+		(at 173.99 182.88 180)
+		(effects
+			(font
+				(size 1.27 1.27)
+			)
+			(justify right bottom)
+		)
+	)
 	(label "USB1.D_P"
 		(at 264.16 101.6 180)
@@
 		)
 	)
+	(label "BT_nDis"
+		(at 173.99 185.42 180)
+		(effects
+			(font
+				(size 1.27 1.27)
+			)
+			(justify right bottom)
+		)
+	)
 	(label "RPI_ETH_G"
 		(at 153.67 40.64 180)
@@
 					(unit 1)
 				)
+			)
+		)
+	)
+	(symbol
+		(lib_id "Connector_Generic:Conn_01x03")
+		(at 133.35 165.1 0)
+		(unit 1)
+		(body_style 1)
+		(exclude_from_sim no)
+		(in_bom yes)
+		(on_board yes)
+		(in_pos_files yes)
+		(dnp no)
+		(fields_autoplaced yes)
+		(property "Reference" "J26"
+			(at 135.89 163.8299 0)
+			(show_name no)
+			(do_not_autoplace no)
+			(effects
+				(font
+					(size 1.27 1.27)
+				)
+				(justify left)
+			)
+		)
+		(property "Value" "Conn_01x03"
+			(at 135.89 166.3699 0)
+			(show_name no)
+			(do_not_autoplace no)
+			(effects
+				(font
+					(size 1.27 1.27)
+				)
+				(justify left)
+			)
+		)
+		(property "Footprint" ""
+			(at 133.35 165.1 0)
+			(hide yes)
+			(show_name no)
+			(do_not_autoplace no)
+			(effects
+				(font
+					(size 1.27 1.27)
+				)
+			)
+		)
+		(property "Datasheet" ""
+			(at 133.35 165.1 0)
+			(hide yes)
+			(show_name no)
+			(do_not_autoplace no)
+			(effects
+				(font
+					(size 1.27 1.27)
+				)
+			)
+		)
+		(property "Description" "Generic connector, single row, 01x03, script generated (kicad-library-utils/schlib/autogen/connector/)"
+			(at 133.35 165.1 0)
+			(hide yes)
+			(show_name no)
+			(do_not_autoplace no)
+			(effects
+				(font
+					(size 1.27 1.27)
+				)
+			)
+		)
+		(pin "1"
+		)
+		(pin "3"
+		)
+		(pin "2"
+		)
+		(instances
+			(project "CMDB_Adv"
+				(path "/e63e39d7-6ac0-4ffd-8aa3-1841a4541b55/40909d69-9b3c-44c1-abea-2634187105ac"
+					(reference "J26")
+					(unit 1)
+				)

Commit message: WIP CMDB-Adv
Parts:
- removed SW2: SW_CONFIG, Button_Switch_SMD:SW_DIP_SPSTx08_Slide_Copal_CHS-08A_W5.08mm_P1.27mm_JPin, symbol Switch:SW_DIP_x08
- added SW2: SW_CONFIG, Button_Switch_SMD:SW_DIP_SPSTx08_Slide_Copal_CHS-08A_W5.08mm_P1.27mm_JPin, symbol Switch:SW_DIP_x06
- J26: value Conn_01x03 -> AUX_BTN; footprint (none) -> Connector_Molex:Molex_PicoBlade_53047-0310_1x03_P1.25mm_Vertical
Connections:
- net BT_nDis: now also SW2.7
- net EEPROM_nWP: now also SW2.11
- net GND: now also J26.3 (Pin_3), SW2.1, SW2.2, SW2.3, SW2.4, SW2.5, SW2.6
- net PMIC_ENABLE: now also J26.2 (Pin_2), SW2.9
- net PWR_BUT: now also J26.1 (Pin_1)
- net USBOTG: now also SW2.10
- net WL_nDis: now also SW2.8
- net nRPIBOOT: now also SW2.12
Other:
- note removed: "TODO: DIP Size"
- moved on the sheet: J19, J26, J5, R11, SW1, TP6, TP7, TP8
