File: pcb_CMDB_Adv/CMDB_Adv.kicad_pcb (KiCad board)
At the start: 6 copper layers, 59.7 x 78 mm, 9 parts, among them J1 POWER TERMINAL, J12 CONN_USB3_A, J13 CONN_USB_PWR_OTG, J15 CONN_DOCK, J16 CONN_CAM1, J17 CONN_CAM0, J2 Bus_M.2_Socket_M, J4 J_PSU_EN

Commit message: CMDB-Adv PCB WIP
Parts:
- removed J1: POWER TERMINAL, CMDB_Adv:Power Terminal
- added H1: MountingHole, CMDB_Adv:MountingHole_2.7mm_M2.5_DIN965, F.Cu at (137.6, 53.4)
- added H2: MountingHole, CMDB_Adv:MountingHole_2.7mm_M2.5_DIN965, F.Cu at (207.4, 53.4)
- added H3: MountingHole, CMDB_Adv:MountingHole_2.7mm_M2.5_DIN965, F.Cu at (207.4, 146.1)
- added H4: MountingHole, CMDB_Adv:MountingHole_2.7mm_M2.5_DIN965, F.Cu at (137.6, 146.1)
- added IC1: KSZ8795CLXCC, CMDB_Adv:QFP40P1200X1200X160-80N, F.Cu at (167.1, 83.7)
- added IC2: Wio-SX1262, CMDB_Adv:Wio-SX1262, F.Cu at (189.9, 133.3)
- added J10: ETH1, CMDB_Adv:CONN12_ARJM11B1-009-AB-EW2_ABR, F.Cu at (198.9, 65.4)
- added J14: CONN_HAT, Connector_PinHeader_2.54mm:PinHeader_2x20_P2.54mm_Vertical, F.Cu at (198.6, 96.9)
- added J18: ETH2, CMDB_Adv:CONN12_ARJM11B1-009-AB-EW2_ABR, F.Cu at (198.9, 84.6)
- added J20: CONN_5VEXT1, Connector_Wire:SolderWirePad_1x01_SMD_3x6mm, F.Cu at (207.1, 131.3)
- added J21: CONN_5VEXT1_GND, Connector_Wire:SolderWirePad_1x01_SMD_3x6mm, F.Cu at (207.1, 127.3)
- added J22: CONN_5VEXT2, Connector_Wire:SolderWirePad_1x01_SMD_3x6mm, F.Cu at (207.1, 140.9)
- added J23: CONN_5VEXT2_GND, Connector_Wire:SolderWirePad_1x01_SMD_3x6mm, F.Cu at (207.1, 136.8)
- added J3: CONN_VIN, Connector_AMASS:AMASS_XT30PW-M_1x02_P2.50mm_Horizontal, F.Cu at (145.9, 131.9)
- added J5: CONN_FAN, Connector_JST:JST_SH_BM04B-SRSS-TB_1x04-1MP_P1.00mm_Vertical, F.Cu at (192.7, 98.5)
- added J6: CONN_UART3, Connector_Molex:Molex_PicoBlade_53048-0310_1x03_P1.25mm_Horizontal, F.Cu at (205.5, 123.1)
- added J7: CONN_SPI, Connector_Molex:Molex_PicoBlade_53048-0610_1x06_P1.25mm_Horizontal, F.Cu at (205.5, 116.5)
- added J8: CONN_I2C, Connector_Molex:Molex_PicoBlade_53048-0310_1x03_P1.25mm_Horizontal, F.Cu at (205.5, 99.5)
- added J9: CONN_UART0, Connector_Molex:Molex_PicoBlade_53048-0310_1x03_P1.25mm_Horizontal, F.Cu at (205.5, 106.1)
- added JP10: ADDR16, Jumper:SolderJumper-3_P2.0mm_Open_TrianglePad1.0x1.5mm, F.Cu at (179.8, 138.2)
- added JP6: ADDR1, Jumper:SolderJumper-3_P2.0mm_Open_TrianglePad1.0x1.5mm, F.Cu at (179.8, 127.0)
- added JP7: ADDR2, Jumper:SolderJumper-3_P2.0mm_Open_TrianglePad1.0x1.5mm, F.Cu at (179.8, 129.8)
- added JP8: ADDR4, Jumper:SolderJumper-3_P2.0mm_Open_TrianglePad1.0x1.5mm, F.Cu at (179.8, 132.6)
- added JP9: ADDR8, Jumper:SolderJumper-3_P2.0mm_Open_TrianglePad1.0x1.5mm, F.Cu at (179.8, 135.4)
- added SW2: SW_CONFIG, Button_Switch_SMD:SW_DIP_SPSTx08_Slide_Copal_CHS-08A_W5.08mm_P1.27mm_JPin, F.Cu at (193.0, 107.3)
- added U5: ESP32-WROOM-32UE, RF_Module:ESP32-WROOM-32UE, B.Cu at (186.2, 130.4)
- added U7: MCP23017_SO, Package_SO:SOIC-28W_7.5x17.9mm_P1.27mm, F.Cu at (182.6, 119.5)
- J4: value J_PSU_EN -> J_ESP_DBG_UART; footprint Connector_PinHeader_2.54mm:PinHeader_1x02_P2.54mm_Vertical -> Connector_Molex:Molex_PicoBlade_53047-0310_1x03_P1.25mm_Vertical
- moved J4 41.5 mm to (194.4, 118.5), turned to 90 degrees
- moved J16 18.7 mm to (139.8, 64.8)
- moved J17 18.7 mm to (139.8, 64.8)
- moved Module1 18.2 mm to (183.6, 59.7)
- moved J15 18.1 mm to (138.8, 85.9)
- moved J12 17.2 mm to (143.7, 108.9)
- moved J2 14.1 mm to (167.0, 73.2)
- moved J13 2.74 mm to (186.5, 147.6)
Connections:
- net /CM5/+5v renamed /+5VPB
- net /CM5/VBAT renamed /CM5/+3V3STB
- net /M2_3V3 renamed /+3V3PB1
- J13 pad A6: /Connectors/USBC.D_P -> /CM5/USBC.D_P
- J13 pad A7: /Connectors/USBC.D_N -> /CM5/USBC.D_N
- J13 pad B6: /Connectors/USBC.D_P -> /CM5/USBC.D_P
- J13 pad B7: /Connectors/USBC.D_N -> /CM5/USBC.D_N
- J15 pad 1: /Connectors/+3.3v -> /Connectors/+5V
- J15 pad 10: unconnected-(J15-Pin_10-Pad10) -> GND
- J15 pad 3: /Connectors/+5v -> /Connectors/+5V
- J15 pad 4: unconnected-(J15-Pin_4-Pad4) -> /CM5/+3V3RPi
- J15 pad 5: unconnected-(J15-Pin_5-Pad5) -> /Connectors/+VBUS_USBA
- J15 pad 7: unconnected-(J15-Pin_7-Pad7) -> /Connectors/+VBUS_USBA
- J15 pad 9: unconnected-(J15-Pin_9-Pad9) -> GND
- J16 pad 22: /Connectors/+3.3v -> /CM5/+3V3RPi
- J17 pad 22: /Connectors/+3.3v -> /CM5/+3V3RPi
- J4 pad 1: /PSU/VIN -> GND
- J4 pad 2: /PSU/PSU_EN -> /Platform Controller/DBG_UART_TX
- Module1 pad 11: GND -> /CM5/ETH0.P2_P
- Module1 pad 35: GND -> /CM5/GPIO1_RAW
- Module1 pad 36: GND -> /CM5/GPIO0_RAW
- Module1 pad 4: GND -> /CM5/ETH0.P1_P
- Module1 pad 41: GND -> /CM5/GP.25
- Module1 pad 51: /CM5/GPIO15_RAW -> /CM5/GP.15
- Module1 pad 55: /CM5/GPIO14_RAW -> /CM5/GP.14
- Module1 pad 6: GND -> /CM5/ETH0.P1_N
- Module1 pad 62: GND -> /CM5/CMD
- Module1 pad 78: /CM5/+3.3v_RPi -> /CM5/+3V3RPi
- Module1 pad 84: /CM5/+3.3v_RPi -> /CM5/+3V3RPi
- Module1 pad 86: /CM5/+3.3v_RPi -> /CM5/+3V3RPi
Routing:
- net /CM5/GP.17: track 0.00 -> 50.2 mm, vias 0 -> 1
- net /CM5/GP.3: track 0.00 -> 44.5 mm, vias 0 -> 1
- net /CM5/GP.2: track 0.00 -> 43.5 mm, vias 0 -> 1
- net /Connectors/GP.27: track 0.00 -> 42.3 mm
- net /CM5/GP.22: track 0.00 -> 41.7 mm
- net /CM5/GP.4: track 0.00 -> 37.0 mm, vias 0 -> 1
- net /CM5/GP.21: track 0.00 -> 36.1 mm
- net /CM5/GP.19: track 0.00 -> 32.7 mm
- net /CM5/GP.20: track 0.00 -> 32.2 mm
- net GND: track 0.00 -> 26.7 mm, vias 6 -> 18
- net /Platform Controller/LORA_RESET: track 0.00 -> 22.6 mm, vias 0 -> 1
- net /Platform Controller/LORA_RF_SW: track 0.00 -> 20.4 mm, vias 0 -> 1
- net /Platform Controller/SPI.SCLK: track 0.00 -> 19.9 mm, vias 0 -> 1
- net /Platform Controller/SPI.MOSI: track 0.00 -> 19.6 mm, vias 0 -> 1
- net /+5VPB: track 0.00 -> 16.4 mm, vias 0 -> 6
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- added copper zone on F.Cu, net /CM5/ETH0.P1_P
- removed copper zone on F.Cu, net GND
Other:
- board size 59.7 x 78 mm -> 76.2 x 99.1 mm
- board text added: "+5VEXT1"
- board text added: "+5VEXT2"
- board text added: "1"
- board text added: "16"
- board text added: "2"
- board text added: "4"
- board text added: "8"
- board text added: "ADDR SEL"
- board text removed: "PSU_EN"
- board text removed: "VIN"

Commit message: CMDB_Adv WIP
Parts:
- added J11: CONN_SDIO, Connector_PinHeader_2.00mm:PinHeader_1x14_P2.00mm_Vertical, B.Cu at (199.1, 51.8)
- added J19: CONN_RTC, Connector_JST:JST_SH_BM02B-SRSS-TB_1x02-1MP_P1.00mm_Vertical, F.Cu at (168.5, 53.0)
- added JP1: GPIO0_SEL, Jumper:SolderJumper-3_P1.3mm_Open_RoundedPad1.0x1.5mm, F.Cu at (185.2, 97.9)
- added JP11: GPIO9_SEL, Jumper:SolderJumper-3_P1.3mm_Open_RoundedPad1.0x1.5mm, F.Cu at (177.3, 84.9)
- added JP2: GPIO1_SEL, Jumper:SolderJumper-3_P1.3mm_Open_RoundedPad1.0x1.5mm, F.Cu at (185.2, 100.9)
- added JP3: ETH_Y_SEL, Jumper:SolderJumper-3_P1.3mm_Open_RoundedPad1.0x1.5mm, F.Cu at (230.9, 88.0)
- added JP4: ETH_G_SEL, Jumper:SolderJumper-3_P1.3mm_Open_RoundedPad1.0x1.5mm, F.Cu at (230.7, 83.6)
- added JP5: GPIO8_SEL, Jumper:SolderJumper-3_P1.3mm_Open_RoundedPad1.0x1.5mm, F.Cu at (177.3, 82.1)
- added SW3: SW_RESET, Button_Switch_SMD:SW_Push_1P1T_NO_CK_KMR2, F.Cu at (173.6, 143.0)
- added SW4: SW_BOOT, Button_Switch_SMD:SW_Push_1P1T_NO_CK_KMR2, F.Cu at (177.3, 143.0)
- added TR1: ALANL100X1-DE12DT, CMDB_Adv:ALANL100X1DE12DT, F.Cu at (174.7, 93.7)
- J2: footprint CMDB_Adv:M.2 M Key socket -> CMDB_Adv:M.2_M_Key_socket_2280
- J6: value CONN_UART3 -> CONN_UART2
- J7: value CONN_SPI -> CONN_SPI1
- J8: value CONN_I2C -> CONN_I2C1
- moved J18 19.4 mm to (199.4, 65.2)
- moved J10 18.9 mm to (199.4, 84.3)
- moved IC1 6.50 mm to (166.9, 77.2), turned to 180 degrees
- moved J2 3.44 mm to (165.4, 70.1)
- moved H2 0.51 mm to (207.5, 52.9)
- moved H1 0.51 mm to (137.6, 52.9)
- moved IC2 0.38 mm to (190.3, 133.3)
- moved J4 0.06 mm to (194.4, 118.5)
Connections:
- net /CM5/ETH0.P2_N renamed /CM5/ETH.P2_N
- net /CM5/ETH0.P2_P renamed /CM5/ETH.P2_P
- net /CM5/ETH0.P3_N renamed /CM5/ETH.P3_N
- net /CM5/ETH0.P3_P renamed /CM5/ETH.P3_P
- net /CM5/PCIe_PWR_EN renamed /+3V3PB1_EN
- net /Connectors/CAM1_GPIO0 renamed /IO Connectors/CAM1_GPIO0
- net /Connectors/ETH1.P0_N renamed /IO Connectors/ETH_DOCK.P0_N
- net /Connectors/ETH1.P0_P renamed /IO Connectors/ETH_DOCK.P0_P
- net /Connectors/ETH1.P1_N renamed /IO Connectors/ETH_DOCK.P1_N
- net /Connectors/ETH1.P1_P renamed /IO Connectors/ETH_DOCK.P1_P
- net /Connectors/ETH1.P2_N renamed /IO Connectors/ETH_DOCK.P2_N
- net /Connectors/ETH1.P2_P renamed /IO Connectors/ETH_DOCK.P2_P
- net /Connectors/ETH1.P3_N renamed /IO Connectors/ETH_DOCK.P3_N
- net /Connectors/ETH1.P3_P renamed /IO Connectors/ETH_DOCK.P3_P
- net /Ethernet/ETH2.RX_N renamed /Eth Switch/ETH2.RX_N
- net /Ethernet/ETH2.RX_P renamed /Eth Switch/ETH2.RX_P
- net /Ethernet/ETH2.TX_N renamed /Eth Switch/ETH2.TX_N
- net /Ethernet/ETH2.TX_P renamed /Eth Switch/ETH2.TX_P
- net /Ethernet/ETH3.RX_N renamed /Eth Switch/ETH3.RX_N
- net /Ethernet/ETH3.RX_P renamed /Eth Switch/ETH3.RX_P
- net /Ethernet/ETH3.TX_N renamed /Eth Switch/ETH3.TX_N
- net /Ethernet/ETH3.TX_P renamed /Eth Switch/ETH3.TX_P
- net /Ethernet/LED1_0 renamed /Eth Switch/ETH1.LED_G
- net /Ethernet/LED1_1 renamed /Eth Switch/ETH1.LED_Y
- net /Ethernet/LED2_0 renamed /Eth Switch/ETH2.LED_G
- net /Ethernet/LED2_1 renamed /Eth Switch/ETH2.LED_Y
- net /Ethernet/LED3_0 renamed Net-(IC1-LED3_0)
- net /Ethernet/LED3_1 renamed Net-(IC1-LED3_1)
- net /Ethernet/LED4_0 renamed /Eth Switch/ETH4.LED_G
- net /Ethernet/LED4_1 renamed /Eth Switch/ETH4.LED_Y
- net /Platform Controller/LORA.CS renamed /Platform Controller/LORA_CS
- net /Platform Controller/RMII.CRS_DV renamed Net-(U5-IO27)
- net /Platform Controller/RMII.RXD0 renamed Net-(U5-IO25)
- net /Platform Controller/RMII.RXD1 renamed Net-(U5-IO26)
- net /Platform Controller/RMII.TXD0 renamed Net-(U5-IO19)
- net /Platform Controller/RMII.TXD1 renamed Net-(U5-IO22)
- net /Platform Controller/RMII.TX_EN renamed Net-(U5-IO21)
- IC1 pad 1: /+1V2PB -> /Eth Switch/+VDD12A
- IC1 pad 12: /+3V3PB2 -> /Eth Switch/+VDDAT
- IC1 pad 17: /Ethernet/ETH4.RX_P -> /Eth Switch/ETH4.RX_P
- IC1 pad 18: /Ethernet/ETH4.RX_N -> /Eth Switch/ETH4.RX_N
- IC1 pad 19: /Ethernet/ETH4.TX_P -> /Eth Switch/ETH4.TX_P
- IC1 pad 2: /+3V3PB2 -> /Eth Switch/+VDDAT
- IC1 pad 20: /Ethernet/ETH4.TX_N -> /Eth Switch/ETH4.TX_N
- IC1 pad 23: unconnected-(IC1-INTR_N-Pad23) -> /Eth Switch/SWITCH_INT
- IC1 pad 26: /+1V2PB -> /Eth Switch/+VDD12D
- IC1 pad 29: unconnected-(IC1-TXEN5/TXDS5_CTL-Pad29) -> /Eth Switch/RMII.TX_EN
- IC1 pad 30: unconnected-(IC1-TXD5_0-Pad30) -> /Eth Switch/RMII.TXD0
- IC1 pad 32: unconnected-(IC1-TXD5_1-Pad32) -> /Eth Switch/RMII.TXD1
- IC1 pad 34: /+3V3PB2 -> /Eth Switch/+VDDIO
- IC1 pad 4: /CM5/ETH0.P0_P -> /Eth Switch/ETH1.RX_P
- IC1 pad 42: /+1V2PB -> /Eth Switch/+VDD12D
- IC1 pad 44: unconnected-(IC1-RXC5/GRXC5-Pad44) -> /Eth Switch/RMII.REFCLK
- IC1 pad 45: unconnected-(IC1-RXD5_0-Pad45) -> /Eth Switch/RMII.RXD0
- IC1 pad 46: unconnected-(IC1-RXD5_1-Pad46) -> /Eth Switch/RMII.RXD1
- IC1 pad 48: /+3V3PB2 -> /Eth Switch/+VDDIO
- IC1 pad 5: /CM5/ETH0.P0_N -> /Eth Switch/ETH1.RX_N
- IC1 pad 51: unconnected-(IC1-RXDV5/CRSDV5/RXD5_CTL-Pad51) -> /Eth Switch/RMII.CRS_DV
- IC1 pad 6: /CM5/ETH0.P1_P -> /Eth Switch/ETH1.TX_P
- IC1 pad 66: /Ethernet/MGMT_SPI.MISO -> /Eth Switch/MGMT_SPI.MISO
- IC1 pad 67: /Ethernet/MGMT_SPI.SCLK -> /Eth Switch/MGMT_SPI.SCLK
- IC1 pad 68: /Ethernet/MGMT_SPI.MOSI -> /Eth Switch/MGMT_SPI.MOSI
- IC1 pad 69: /Ethernet/MGMT_SPI.CS -> /Eth Switch/MGMT_SPI.CS
- IC1 pad 7: /CM5/ETH0.P1_N -> /Eth Switch/ETH1.TX_N
- IC1 pad 70: /+3V3PB2 -> /Eth Switch/+VDDIO
- IC1 pad 72: /Ethernet/RST_N -> /Eth Switch/RST_N
- IC1 pad 73: /+1V2PB -> /Eth Switch/+VDD12D
- IC1 pad 76: /+3V3PB2 -> /Eth Switch/+VDDAT
- IC1 pad 79: unconnected-(IC1-XI-Pad79) -> Net-(IC1-XI)
- IC2 pad 2: /Platform Controller/SPI.MISO -> /Eth Switch/MGMT_SPI.MISO
- IC2 pad 3: /Platform Controller/SPI.MOSI -> /Eth Switch/MGMT_SPI.MOSI
- IC2 pad 4: /Platform Controller/SPI.SCLK -> /Eth Switch/MGMT_SPI.SCLK
- J10 pad 1: /CM5/ETH0.P1_P -> /Eth Switch/ETH1.TX_P
- J10 pad 2: /CM5/ETH0.P1_N -> /Eth Switch/ETH1.TX_N
- J10 pad 3: /CM5/ETH0.P0_P -> /Eth Switch/ETH1.RX_P
- J10 pad 6: /CM5/ETH0.P0_N -> /Eth Switch/ETH1.RX_N
- J10 pad SH: GND -> Net-(J10-PadSH)
- J12 pad 1: /Connectors/+VBUS_USBA -> /IO Connectors/+VBUS_USBA
- J12 pad 10: GND -> (no net)
- J12 pad 2: /CM5/USB1.RX_N -> /CM5/USB1.D_N
- J12 pad 3: /CM5/USB1.RX_P -> /CM5/USB1.D_P
- J12 pad 5: /CM5/USB1.D_P -> /CM5/USB1.RX_N
- J12 pad 6: /CM5/USB1.D_N -> /CM5/USB1.RX_P
- J13 pad A1_B12: (no net) -> GND
- J13 pad A4_B9: (no net) -> /+VBUS_USBC
- J13 pad A5: /Connectors/CC1 -> /CM5/USBC.CC1
- J13 pad B1_A12: (no net) -> GND
- J13 pad B4_A9: (no net) -> /+VBUS_USBC
- J13 pad B5: /Connectors/CC2 -> /CM5/USBC.CC2
- J13 pad S2: (no net) -> GND
- J13 pad S3: (no net) -> GND
- J13 pad S4: (no net) -> GND
- J14 pad 13: /Connectors/GP.27 -> /CM5/GP.27
- J14 pad 2: /Connectors/+5V -> /+5VPB
- J14 pad 4: /Connectors/+5V -> /+5VPB
- J15 pad 1: /Connectors/+5V -> /+5VPB
- J15 pad 2: GND -> /IO Connectors/+VBUS_USBA
- J15 pad 3: /Connectors/+5V -> /+5VPB
- J15 pad 4: /CM5/+3V3RPi -> /IO Connectors/+VBUS_USBA
- J15 pad 5: /Connectors/+VBUS_USBA -> /IO Connectors/PCTL_DBG_UART_TX
- J15 pad 6: unconnected-(J15-Pin_6-Pad6) -> /CM5/+3V3RPi
- J15 pad 7: /Connectors/+VBUS_USBA -> /IO Connectors/PCTL_DBG_UART_RX
- J15 pad 8: unconnected-(J15-Pin_8-Pad8) -> GND
- J18 pad SH: GND -> Net-(J18-PadSH)
- J4 pad 2: /Platform Controller/DBG_UART_TX -> /IO Connectors/PCTL_DBG_UART_TX
- J4 pad 3: /Platform Controller/DBG_UART_RX -> /IO Connectors/PCTL_DBG_UART_RX
- J5 pad 1: /CM5/+5v -> /+5VPB
- J6 pad 1: /CM5/GP.8 -> /CM5/GP.4
- J6 pad 2: /CM5/GP.9 -> /CM5/GP.5
- Module1 pad 10: /CM5/ETH0.P0_N -> /CM5/ETH.P0_N
- Module1 pad 12: /CM5/ETH0.P0_P -> /CM5/ETH.P0_P
- Module1 pad 15: unconnected-(Module1A-Ethernet_nLED3(3.3v)-Pad15) -> /CM5/RPI_ETH_G
- Module1 pad 17: unconnected-(Module1A-Ethernet_nLED2(3.3v)-Pad17) -> /CM5/RPI_ETH_Y
- Module1 pad 18: /CM5/SYNC_OUT -> unconnected-(Module1A-Ethernet_SYNC_OUT(3.3v)-Pad18)
- Module1 pad 39: /CM5/GP.8 -> /CM5/GPIO8_RAW
- Module1 pad 4: /CM5/ETH0.P1_P -> /CM5/ETH.P1_P
- Module1 pad 40: /CM5/GP.9 -> /CM5/GPIO9_RAW
- Module1 pad 6: /CM5/ETH0.P1_N -> /CM5/ETH.P1_N
- Module1 pad 62: /CM5/CMD -> /CM5/SD.CMD
- Module1 pad 64: unconnected-(Module1A-SD_DAT5-Pad64) -> /CM5/SD.DAT5
- Module1 pad 68: unconnected-(Module1A-SD_DAT4-Pad68) -> /CM5/SD.DAT4
- Module1 pad 70: unconnected-(Module1A-SD_DAT7-Pad70) -> /CM5/SD.DAT7
- Module1 pad 72: unconnected-(Module1A-SD_DAT6-Pad72) -> /CM5/SD.DAT6
- SW2 pad 10: unconnected-(SW2-Pad10) -> /CM5/WL_nDis
- SW2 pad 14: /CM5/SYNC_OUT -> unconnected-(SW2-Pad14)
- SW2 pad 8: /CM5/+3.3v_STDB -> GND
- SW2 pad 9: /CM5/VBAT -> /CM5/BT_nDis
- U5 pad 23: /Platform Controller/UART_TX -> /CM5/UART_PCTL_RX
- U5 pad 26: /Platform Controller/SWITCH_RST_N -> /Eth Switch/RST_N
- U5 pad 28: /Platform Controller/SPI.MOSI -> /Eth Switch/MGMT_SPI.MOSI
- U5 pad 30: /Platform Controller/SPI.SCLK -> /Eth Switch/MGMT_SPI.SCLK
- U5 pad 34: /Platform Controller/DBG_UART_RX -> /IO Connectors/PCTL_DBG_UART_RX
- U5 pad 35: /Platform Controller/DBG_UART_TX -> /IO Connectors/PCTL_DBG_UART_TX
- U5 pad 4: /Platform Controller/UART_RX -> /CM5/UART_PCTL_TX
- U5 pad 5: unconnected-(U5-SENSOR_VN-Pad5) -> /Eth Switch/SWITCH_INT
- U5 pad 7: /Platform Controller/SPI.MISO -> /Eth Switch/MGMT_SPI.MISO
- U5 pad 9: /Platform Controller/SWITCH.CS -> /Eth Switch/MGMT_SPI.CS
- U7 pad 1: /Platform Controller/ADDR1 -> /+5VPB_EN
- U7 pad 2: /Platform Controller/ADDR2 -> /+5VEXT1_EN
- U7 pad 21: unconnected-(U7-GPA0-Pad21) -> /Platform Controller/ADDR1
- U7 pad 22: unconnected-(U7-GPA1-Pad22) -> /Platform Controller/ADDR2
- U7 pad 23: unconnected-(U7-GPA2-Pad23) -> /Platform Controller/ADDR4
- U7 pad 24: unconnected-(U7-GPA3-Pad24) -> /Platform Controller/ADDR8
- U7 pad 25: unconnected-(U7-GPA4-Pad25) -> /Platform Controller/ADDR16
- U7 pad 26: unconnected-(U7-GPA5-Pad26) -> /Platform Controller/LED_ACT
- U7 pad 3: /Platform Controller/ADDR4 -> /+5VEXT2_EN
- U7 pad 4: /Platform Controller/ADDR8 -> unconnected-(U7-GPB3-Pad4)
- U7 pad 5: /Platform Controller/ADDR16 -> unconnected-(U7-GPB4-Pad5)
- U7 pad 6: /Platform Controller/LED_ACT -> unconnected-(U7-GPB5-Pad6)
Routing:
- net /CM5/GP.16: track 0.00 -> 78.4 mm, vias 0 -> 1
- net /CM5/GP.26: track 0.00 -> 71.8 mm, vias 0 -> 1
- net /CM5/GP.8: track 5.04 -> 75.7 mm, vias 0 -> 1
- net /CM5/GP.19: track 32.7 -> 103.0 mm, vias 0 -> 1
- net /CM5/GP.12: track 0.00 -> 68.9 mm, vias 0 -> 1
- net /CM5/GP.13: track 0.00 -> 65.1 mm, vias 0 -> 1
- net /CM5/GP.6: track 0.00 -> 64.8 mm, vias 0 -> 1
- net /CM5/GP.7: track 0.00 -> 60.4 mm, vias 0 -> 1
- net /CM5/GP.5: track 0.00 -> 60.3 mm, vias 0 -> 1
- net /CM5/GP.1: track 0.00 -> 58.1 mm, vias 0 -> 1
- net /Eth Switch/ETH1.TX_N: track 0.00 -> 57.1 mm
- net /Eth Switch/ETH1.TX_P: track 0.00 -> 57.0 mm
- net /CM5/GP.11: track 0.00 -> 54.9 mm, vias 0 -> 1
- net /CM5/GP.25: track 0.00 -> 53.6 mm, vias 0 -> 1
- net /CM5/GP.9: track 7.52 -> 59.2 mm, vias 0 -> 1
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- added copper zone on F.Cu, net /CM5/ETH.P1_P
- removed copper zone on F.Cu, net /CM5/ETH0.P1_P
Other:
- board size 76.2 x 99.1 mm -> 76.2 x 99.4 mm
- board text added: "TODO: CONSIDER ADDING GND FILL TO UPER LAYERS FOR THERMAL PROPERTIES"

Commit message: WIP
Parts:
- moved J13 54.0 mm to (136.0, 128.4), turned to -90 degrees
- moved J3 5.84 mm to (145.4, 137.7), turned to 180 degrees
- moved SW4 3.99 mm to (181.3, 143.2)
- moved SW3 3.99 mm to (177.6, 143.2)
- moved J12 1.58 mm to (143.8, 110.5)
Routing:
- net /CM5/MIPI0.D0_N: track 0.00 -> 63.0 mm, vias 0 -> 2
- net /CM5/MIPI0.D0_P: track 0.00 -> 63.0 mm, vias 0 -> 2
- net /CM5/MIPI0.D2_N: track 0.00 -> 62.9 mm, vias 0 -> 2
- net /CM5/MIPI0.D2_P: track 0.00 -> 62.9 mm, vias 0 -> 2
- net /CM5/MIPI0.D1_P: track 0.00 -> 62.6 mm, vias 0 -> 2
- net /CM5/MIPI0.D1_N: track 0.00 -> 62.6 mm, vias 0 -> 2
- net /CM5/MIPI0.CK_P: track 0.00 -> 62.2 mm, vias 0 -> 2
- net /CM5/MIPI0.CK_N: track 0.00 -> 62.2 mm, vias 0 -> 2
- net /CM5/MIPI0.D3_P: track 0.00 -> 60.3 mm, vias 0 -> 2
- net /CM5/MIPI0.D3_N: track 0.00 -> 60.3 mm, vias 0 -> 2
- net /CM5/USBC.D_P: track 0.00 -> 50.2 mm, vias 0 -> 2
- net /CM5/USBC.D_N: track 0.00 -> 48.9 mm, vias 0 -> 2
- net /CM5/USB1.RX_N: track 0.00 -> 47.8 mm, vias 0 -> 1
- net /CM5/USB1.RX_P: track 0.00 -> 47.8 mm, vias 0 -> 1
- net /CM5/USB1.D_P: track 0.00 -> 46.3 mm, vias 0 -> 2
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- added copper zone on F.Cu, net /+VBUS_USBC
- added copper zone on F.Cu, net GND
Other:
- outline, holes or cut-outs redrawn
- board text removed: "100R"
- board text removed: "90R"

Commit message: WIP CMDB-Adv
Parts:
- added C18: 100n, Capacitor_SMD:C_0805_2012Metric_Pad1.18x1.45mm_HandSolder, F.Cu at (77.8, 64.3)
- added C19: 10u, Capacitor_SMD:C_0805_2012Metric_Pad1.18x1.45mm_HandSolder, F.Cu at (72.0, 84.0)
- added C20: 100uF, Capacitor_Tantalum_SMD:CP_EIA-7343-31_Kemet-D, B.Cu at (138.6, 106.8)
- added C21: 10u, Capacitor_SMD:C_0805_2012Metric_Pad1.18x1.45mm_HandSolder, F.Cu at (72.0, 87.0)
- added C22: 10u, Capacitor_SMD:C_0805_2012Metric_Pad1.18x1.45mm_HandSolder, F.Cu at (72.0, 90.0)
- added C23: 100n, Capacitor_SMD:C_0805_2012Metric_Pad1.18x1.45mm_HandSolder, F.Cu at (77.8, 67.3)
- added C24: 100n, Capacitor_SMD:C_0805_2012Metric_Pad1.18x1.45mm_HandSolder, F.Cu at (77.8, 70.3)
- added C25: 100n, Capacitor_SMD:C_0805_2012Metric_Pad1.18x1.45mm_HandSolder, F.Cu at (77.8, 73.3)
- added C27: 100nF, Capacitor_SMD:C_0402_1005Metric_Pad0.74x0.62mm_HandSolder, F.Cu at (63.8, 63.8)
- added C28: 100nF, Capacitor_SMD:C_0402_1005Metric_Pad0.74x0.62mm_HandSolder, F.Cu at (63.8, 65.7)
- added C29: 100nF, Capacitor_SMD:C_0402_1005Metric_Pad0.74x0.62mm_HandSolder, F.Cu at (63.8, 67.7)
- added C3: 100n, Capacitor_SMD:C_0805_2012Metric_Pad1.18x1.45mm_HandSolder, F.Cu at (73.3, 111.8)
- added C30: 22uF, Capacitor_SMD:C_1206_3216Metric_Pad1.33x1.80mm_HandSolder, F.Cu at (59.2, 64.4)
- added C31: 22uF, Capacitor_SMD:C_1206_3216Metric_Pad1.33x1.80mm_HandSolder, F.Cu at (59.2, 67.8)
- added C32: 100nF, Capacitor_SMD:C_0402_1005Metric_Pad0.74x0.62mm_HandSolder, F.Cu at (63.8, 69.7)
- added C33: 100nF, Capacitor_SMD:C_0402_1005Metric_Pad0.74x0.62mm_HandSolder, F.Cu at (63.8, 71.6)
- added C34: 100nF, Capacitor_SMD:C_0402_1005Metric_Pad0.74x0.62mm_HandSolder, F.Cu at (63.8, 73.6)
- added C35: 22uF, Capacitor_SMD:C_1206_3216Metric_Pad1.33x1.80mm_HandSolder, F.Cu at (59.2, 71.1)
- added C36: 100nF, Capacitor_SMD:C_0402_1005Metric_Pad0.74x0.62mm_HandSolder, F.Cu at (67.1, 63.8)
- added C37: 100nF, Capacitor_SMD:C_0402_1005Metric_Pad0.74x0.62mm_HandSolder, F.Cu at (67.1, 65.7)
- added C38: 100nF, Capacitor_SMD:C_0402_1005Metric_Pad0.74x0.62mm_HandSolder, F.Cu at (67.1, 67.7)
- added C39: 22uF, Capacitor_SMD:C_1206_3216Metric_Pad1.33x1.80mm_HandSolder, F.Cu at (59.2, 74.5)
- added C40: 100nF, Capacitor_SMD:C_0402_1005Metric_Pad0.74x0.62mm_HandSolder, F.Cu at (67.1, 69.7)
- added C42: 100nF, Capacitor_SMD:C_0402_1005Metric_Pad0.74x0.62mm_HandSolder, F.Cu at (67.1, 71.6)
- added C43: 22uF, Capacitor_SMD:C_1206_3216Metric_Pad1.33x1.80mm_HandSolder, F.Cu at (35.9, 95.8)
- added C44: 100nF, Capacitor_SMD:C_0402_1005Metric_Pad0.74x0.62mm_HandSolder, F.Cu at (34.5, 105.2)
- added C45: 100nF, Capacitor_SMD:C_0402_1005Metric_Pad0.74x0.62mm_HandSolder, F.Cu at (42.6, 95.1)
- added C46: 100nF, Capacitor_SMD:C_0402_1005Metric_Pad0.74x0.62mm_HandSolder, F.Cu at (42.6, 97.1)
- added C47: 100nF, Capacitor_SMD:C_0402_1005Metric_Pad0.74x0.62mm_HandSolder, F.Cu at (42.6, 99.0)
- added C48: 100nF, Capacitor_SMD:C_0402_1005Metric_Pad0.74x0.62mm_HandSolder, F.Cu at (42.6, 101.0)
- added C49: 22uF, Capacitor_SMD:C_1206_3216Metric_Pad1.33x1.80mm_HandSolder, F.Cu at (35.9, 99.1)
- added C50: 100nF, Capacitor_SMD:C_0402_1005Metric_Pad0.74x0.62mm_HandSolder, F.Cu at (34.5, 107.1)
- added C51: 100nF, Capacitor_SMD:C_0402_1005Metric_Pad0.74x0.62mm_HandSolder, F.Cu at (34.5, 109.1)
- added C52: 100nF, Capacitor_SMD:C_0402_1005Metric_Pad0.74x0.62mm_HandSolder, F.Cu at (34.5, 111.1)
- added C53: 10uF, Capacitor_SMD:C_1206_3216Metric_Pad1.33x1.80mm_HandSolder, F.Cu at (35.9, 102.5)
- added C54: 100nF, Capacitor_SMD:C_0402_1005Metric_Pad0.74x0.62mm_HandSolder, F.Cu at (42.9, 63.8)
- added C55: 100nF, Capacitor_SMD:C_0402_1005Metric_Pad0.74x0.62mm_HandSolder, F.Cu at (42.9, 65.7)
- added C57: 100nF, Capacitor_SMD:C_0402_1005Metric_Pad0.74x0.62mm_HandSolder, F.Cu at (42.9, 67.7)
- added C58: 22uF, Capacitor_SMD:C_1206_3216Metric_Pad1.33x1.80mm_HandSolder, F.Cu at (169.9, 68.0)
- added C59: 100nF, Capacitor_SMD:C_0402_1005Metric_Pad0.74x0.62mm_HandSolder, F.Cu at (42.9, 69.7)
- added C62: 100nF, Capacitor_SMD:C_0402_1005Metric_Pad0.74x0.62mm_HandSolder, F.Cu at (59.6, 93.5)
- added C63: 100nF, Capacitor_SMD:C_0402_1005Metric_Pad0.74x0.62mm_HandSolder, F.Cu at (42.9, 71.6)
- added C64: 100nF, Capacitor_SMD:C_0402_1005Metric_Pad0.74x0.62mm_HandSolder, F.Cu at (59.6, 95.5)
- added C65: 10uF, Capacitor_SMD:C_1206_3216Metric_Pad1.33x1.80mm_HandSolder, F.Cu at (21.7, 64.4)
- added C66: 10uF, Capacitor_SMD:C_1206_3216Metric_Pad1.33x1.80mm_HandSolder, F.Cu at (21.7, 67.8)
- added C67: 10uF, Capacitor_SMD:C_1206_3216Metric_Pad1.33x1.80mm_HandSolder, F.Cu at (21.7, 71.1)
- added C68: 10uF, Capacitor_SMD:C_1206_3216Metric_Pad1.33x1.80mm_HandSolder, F.Cu at (21.7, 74.5)
- added C69: 10uF, Capacitor_SMD:C_1206_3216Metric_Pad1.33x1.80mm_HandSolder, F.Cu at (21.7, 77.8)
- added C70: 10uF, Capacitor_SMD:C_1206_3216Metric_Pad1.33x1.80mm_HandSolder, F.Cu at (21.7, 81.2)
- added C72: 22uF, Capacitor_SMD:C_1206_3216Metric_Pad1.33x1.80mm_HandSolder, F.Cu at (172.3, 68.0)
- added C73: 22uF, Capacitor_SMD:C_1206_3216Metric_Pad1.33x1.80mm_HandSolder, B.Cu at (179.5, 65.7)
- added C8: 470nF, Capacitor_SMD:C_0805_2012Metric_Pad1.18x1.45mm_HandSolder, F.Cu at (26.0, 110.4)
- added D1: LED Green, LED_SMD:LED_0603_1608Metric, F.Cu at (72.9, 106.4)
- added D10: PWR_VALID, Diode_SMD:D_0805_2012Metric_Pad1.15x1.40mm_HandSolder, F.Cu at (34.2, 64.3)
- added D11: +5VPB, Diode_SMD:D_0805_2012Metric_Pad1.15x1.40mm_HandSolder, F.Cu at (34.2, 67.3)
- added D12: ETH4_Y, LED_SMD:LED_0603_1608Metric_Pad1.05x0.95mm_HandSolder, F.Cu at (77.7, 76.1)
- added D13: +5VEXT1, Diode_SMD:D_0805_2012Metric_Pad1.15x1.40mm_HandSolder, F.Cu at (34.2, 70.4)
- added D14: +5VEXT2, Diode_SMD:D_0805_2012Metric_Pad1.15x1.40mm_HandSolder, F.Cu at (34.2, 73.4)
- added D15: BAT54A, Package_TO_SOT_SMD:SOT-23, F.Cu at (21.1, 111.1)
- added D16: +VIMM, Diode_SMD:D_0805_2012Metric_Pad1.15x1.40mm_HandSolder, F.Cu at (34.2, 76.4)
- added D17: ETH4_G, LED_SMD:LED_0603_1608Metric_Pad1.05x0.95mm_HandSolder, F.Cu at (77.7, 78.7)
- added D2: SS34, Diode_SMD:D_SMA_Handsoldering, F.Cu at (115.4, 119.8)
- added D3: LED Red, LED_SMD:LED_0603_1608Metric, F.Cu at (72.9, 109.0)
- added D4: GREEN, LED_SMD:LED_0603_1608Metric, F.Cu at (57.4, 101.7)
- added D5: RED, LED_SMD:LED_0603_1608Metric, F.Cu at (57.4, 104.3)
- added D6: GREEN, LED_SMD:LED_0603_1608Metric, F.Cu at (57.4, 106.9)
- added D7: AMBER, LED_SMD:LED_0603_1608Metric, F.Cu at (57.4, 109.5)
- added D8: LED Green, LED_SMD:LED_0603_1608Metric, F.Cu at (30.4, 110.2)
- added D9: SS34, Diode_SMD:D_SMA_Handsoldering, F.Cu at (115.4, 124.4)
- added FB1: BLM21PG221SN1D, Inductor_SMD:L_0805_2012Metric_Pad1.05x1.20mm_HandSolder, F.Cu at (53.8, 64.1)
- added FB2: BLM21PG221SN1D, Inductor_SMD:L_0805_2012Metric_Pad1.05x1.20mm_HandSolder, F.Cu at (53.8, 66.9)
- added FB3: BLM21PG221SN1D, Inductor_SMD:L_0805_2012Metric_Pad1.05x1.20mm_HandSolder, F.Cu at (53.8, 69.6)
- added FB4: BLM21PG221SN1D, Inductor_SMD:L_0805_2012Metric_Pad1.05x1.20mm_HandSolder, F.Cu at (53.8, 72.4)
- added FB5: BLM21PG221SN1D, Inductor_SMD:L_0805_2012Metric_Pad1.05x1.20mm_HandSolder, F.Cu at (53.8, 75.1)
- added J24: AUX_PWR_OUT1, Connector_PinSocket_2.00mm:PinSocket_2x04_P2.00mm_Vertical, F.Cu at (159.9, 139.6)
- added J25: PL_CTRL_IO, Connector_PinSocket_2.00mm:PinSocket_2x06_P2.00mm_Vertical, F.Cu at (177.1, 144.5)
- added J27: AUX_PWR_OUT2, Connector_PinSocket_2.00mm:PinSocket_2x04_P2.00mm_Vertical, F.Cu at (138.8, 116.7)
- added JP12: +3V3PB2 DIS, Jumper:SolderJumper-3_P1.3mm_Bridged12_RoundedPad1.0x1.5mm, F.Cu at (39.5, 80.5)
- added JP13: +3V3PB3 DIS, Jumper:SolderJumper-3_P1.3mm_Bridged12_RoundedPad1.0x1.5mm, F.Cu at (39.5, 84.3)
- added JP14: +1V2PB DIS, Jumper:SolderJumper-3_P1.3mm_Bridged12_RoundedPad1.0x1.5mm, F.Cu at (39.5, 88.2)
- added Q1: AON7534, Package_DFN_QFN:DFN-8-1EP_3x3mm_P0.65mm_EP1.6x2.56mm_ThermalVias, F.Cu at (27.7, 82.8)
- added Q2: AON7534, Package_DFN_QFN:DFN-8-1EP_3x3mm_P0.65mm_EP1.6x2.56mm_ThermalVias, F.Cu at (27.7, 87.3)
- added R1: 1K, Resistor_SMD:R_0805_2012Metric_Pad1.20x1.40mm_HandSolder, F.Cu at (73.2, 100.7)
- added R10: 1K, Resistor_SMD:R_0805_2012Metric_Pad1.20x1.40mm_HandSolder, F.Cu at (48.9, 110.7)
- added R11: 10K, Resistor_SMD:R_0805_2012Metric_Pad1.20x1.40mm_HandSolder, F.Cu at (48.9, 113.7)
- added R13: 1K, Resistor_SMD:R_0805_2012Metric_Pad1.20x1.40mm_HandSolder, F.Cu at (21.1, 95.6)
- added R14: 4K7, Resistor_SMD:R_0805_2012Metric_Pad1.20x1.40mm_HandSolder, F.Cu at (21.1, 98.5)
- added R15: 4K7, Resistor_SMD:R_0805_2012Metric_Pad1.20x1.40mm_HandSolder, F.Cu at (21.1, 101.5)
- added R16: 2.2K, Resistor_SMD:R_0805_2012Metric_Pad1.20x1.40mm_HandSolder, F.Cu at (67.2, 83.9)
- added R17: 15K, Resistor_SMD:R_0805_2012Metric_Pad1.20x1.40mm_HandSolder, F.Cu at (67.2, 86.9)
- added R18: 2.2K, Resistor_SMD:R_0805_2012Metric_Pad1.20x1.40mm_HandSolder, F.Cu at (67.2, 89.8)
- added R19: 2.2K, Resistor_SMD:R_0805_2012Metric_Pad1.20x1.40mm_HandSolder, F.Cu at (67.2, 92.8)
- added R2: 1K, Resistor_SMD:R_0805_2012Metric_Pad1.20x1.40mm_HandSolder, F.Cu at (73.2, 103.6)
- added R20: 2.2K, Resistor_SMD:R_0805_2012Metric_Pad1.20x1.40mm_HandSolder, F.Cu at (67.2, 95.7)
- added R21: 1K, Resistor_SMD:R_0805_2012Metric_Pad1.20x1.40mm_HandSolder, F.Cu at (21.1, 104.4)
- added R22: 22R, Resistor_SMD:R_0402_1005Metric_Pad0.72x0.64mm_HandSolder, B.Cu at (178.1, 119.5)
- added R24: 2K2, Resistor_SMD:R_0805_2012Metric_Pad1.20x1.40mm_HandSolder, F.Cu at (25.8, 95.6)
- added R25: 2K2, Resistor_SMD:R_0805_2012Metric_Pad1.20x1.40mm_HandSolder, F.Cu at (25.8, 98.5)
- added R26: 1K, Resistor_SMD:R_0805_2012Metric_Pad1.20x1.40mm_HandSolder, F.Cu at (39.0, 64.2)
- added R27: 220R, Resistor_SMD:R_0805_2012Metric_Pad1.20x1.40mm_HandSolder, F.Cu at (73.1, 64.2)
- added R28: 12K4 1%, Resistor_SMD:R_0805_2012Metric_Pad1.20x1.40mm_HandSolder, F.Cu at (48.9, 64.2)
- added R29: 1K, Resistor_SMD:R_0805_2012Metric_Pad1.20x1.40mm_HandSolder, F.Cu at (39.0, 67.2)
- added R30: 1K, Resistor_SMD:R_0805_2012Metric_Pad1.20x1.40mm_HandSolder, F.Cu at (39.0, 70.1)
- added R32: 1K, Resistor_SMD:R_0805_2012Metric_Pad1.20x1.40mm_HandSolder, F.Cu at (39.0, 73.1)
- added R33: 330R, Resistor_SMD:R_0805_2012Metric_Pad1.20x1.40mm_HandSolder, F.Cu at (48.9, 67.2)
- added R34: 1K, Resistor_SMD:R_0805_2012Metric_Pad1.20x1.40mm_HandSolder, F.Cu at (48.9, 70.1)
- added R35: 220R, Resistor_SMD:R_0805_2012Metric_Pad1.20x1.40mm_HandSolder, F.Cu at (73.1, 67.2)
- added R36: 220R, Resistor_SMD:R_0805_2012Metric_Pad1.20x1.40mm_HandSolder, F.Cu at (73.1, 70.1)
- added R37: 220R, Resistor_SMD:R_0805_2012Metric_Pad1.20x1.40mm_HandSolder, F.Cu at (73.1, 73.1)
- added R38: 4K7, Resistor_SMD:R_0805_2012Metric_Pad1.20x1.40mm_HandSolder, F.Cu at (48.9, 73.1)
- added R39: 1K, Resistor_SMD:R_0805_2012Metric_Pad1.20x1.40mm_HandSolder, F.Cu at (48.9, 76.0)
- added R41: 1K, Resistor_SMD:R_0805_2012Metric_Pad1.20x1.40mm_HandSolder, F.Cu at (48.9, 79.0)
- added R42: 1K, Resistor_SMD:R_0805_2012Metric_Pad1.20x1.40mm_HandSolder, F.Cu at (73.1, 76.0)
- added R43: 1K, Resistor_SMD:R_0805_2012Metric_Pad1.20x1.40mm_HandSolder, F.Cu at (73.1, 79.0)
- added R44: 10K, Resistor_SMD:R_0805_2012Metric_Pad1.20x1.40mm_HandSolder, F.Cu at (25.8, 101.5)
- added R46: 1K, Resistor_SMD:R_0805_2012Metric_Pad1.20x1.40mm_HandSolder, F.Cu at (55.6, 94.0)
- added R47: 1K, Resistor_SMD:R_0805_2012Metric_Pad1.20x1.40mm_HandSolder, F.Cu at (55.6, 96.9)
- added R52: 22R, Resistor_SMD:R_0402_1005Metric_Pad0.72x0.64mm_HandSolder, B.Cu at (185.7, 119.6)
- added R53: 22R, Resistor_SMD:R_0402_1005Metric_Pad0.72x0.64mm_HandSolder, B.Cu at (188.2, 119.5)
- added R54: 22R, Resistor_SMD:R_0402_1005Metric_Pad0.72x0.64mm_HandSolder, B.Cu at (192.0, 119.5)
- added R55: 22R, Resistor_SMD:R_0402_1005Metric_Pad0.72x0.64mm_HandSolder, B.Cu at (183.1, 141.4)
- added R56: 22R, Resistor_SMD:R_0402_1005Metric_Pad0.72x0.64mm_HandSolder, B.Cu at (181.9, 141.3)
- added R57: 22R, Resistor_SMD:R_0402_1005Metric_Pad0.72x0.64mm_HandSolder, B.Cu at (180.6, 141.3)
- added R58: 1K, Resistor_SMD:R_0805_2012Metric_Pad1.20x1.40mm_HandSolder, F.Cu at (39.0, 76.0)
- added R7: 1K, Resistor_SMD:R_0805_2012Metric_Pad1.20x1.40mm_HandSolder, F.Cu at (48.9, 101.9)
- added R8: 1K, Resistor_SMD:R_0805_2012Metric_Pad1.20x1.40mm_HandSolder, F.Cu at (48.9, 104.8)
- added R9: 1K, Resistor_SMD:R_0805_2012Metric_Pad1.20x1.40mm_HandSolder, F.Cu at (48.9, 107.8)
- added SW1: BT_PWR, Button_Switch_SMD:SW_Push_1P1T_NO_CK_KMR2, F.Cu at (138.0, 126.4)
- added TP10: TP VBUS_USB, TestPoint:TestPoint_Pad_2.0x2.0mm, F.Cu at (76.4, 84.5)
- added TP13: PWR_VALID1, TestPoint:TestPoint_Pad_1.5x1.5mm, F.Cu at (61.1, 87.8)
- added TP5: PWR_VALID0, TestPoint:TestPoint_Pad_1.5x1.5mm, F.Cu at (61.1, 84.2)
- added TP6: +3V3 RPi, TestPoint:TestPoint_Pad_2.0x2.0mm, F.Cu at (53.3, 102.4)
- added TP7: TP nPWR, TestPoint:TestPoint_Pad_2.0x2.0mm, F.Cu at (53.3, 106.5)
- added TP8: TP nACT, TestPoint:TestPoint_Pad_2.0x2.0mm, F.Cu at (53.3, 110.5)
- added U1: ASEK-32.768KHZ-L-R-T, Crystal:Crystal_SMD_3225-4Pin_3.2x2.5mm, F.Cu at (67.5, 111.5)
- added U10: INA3221, Package_DFN_QFN:Texas_RGV0016A_VQFN-16-1EP_4x4mm_P0.65mm_EP2.1x2.1mm, F.Cu at (50.1, 85.6)
- added U11: INA3221, Package_DFN_QFN:Texas_RGV0016A_VQFN-16-1EP_4x4mm_P0.65mm_EP2.1x2.1mm, F.Cu at (50.1, 91.9)
- added U2: LM74700, Package_TO_SOT_SMD:SOT-23-6, F.Cu at (21.3, 85.3)
- added U3: LM74700, Package_TO_SOT_SMD:SOT-23-6, F.Cu at (21.3, 89.9)
- added U4: TPS7A91, Package_DFN_QFN:Texas_S-PDSO-N10_EP1.2x2mm, F.Cu at (34.6, 80.0)
- added U6: AP22653W6, Package_TO_SOT_SMD:SOT-23-6, F.Cu at (72.2, 93.9)
- added U8: TPS7A91, Package_DFN_QFN:Texas_S-PDSO-N10_EP1.2x2mm, F.Cu at (34.6, 84.0)
- added U9: TPS7A91, Package_DFN_QFN:Texas_S-PDSO-N10_EP1.2x2mm, F.Cu at (34.6, 88.1)
- added Y1: ASE-25.000MHZ-LC-T, Oscillator:Oscillator_SMD_Abracon_ASE-4Pin_3.2x2.5mm, F.Cu at (171.0, 86.0)
- moved JP4 93.3 mm to (143.0, 51.6)
- moved JP3 90.7 mm to (147.9, 51.6)
- moved SW3 16.8 mm to (194.3, 144.8)
- moved SW4 9.50 mm to (190.7, 144.8)
- moved J13 7.32 mm to (136.0, 135.7)
- moved J12 6.76 mm to (143.8, 103.7)
- moved TR1 1.85 mm to (174.8, 95.6)
- moved J3 1.34 mm to (146.7, 137.6)
Connections:
- net /Eth Switch/ETH4.LED_G renamed /ETH.LED_G
- net /Eth Switch/ETH4.LED_Y renamed /ETH.LED_Y
- IC1 pad 13: /Eth Switch/ETH3.RX_P -> /ETH3.RX_P
- IC1 pad 14: /Eth Switch/ETH3.RX_N -> /ETH3.RX_N
- IC1 pad 15: /Eth Switch/ETH3.TX_P -> /ETH3.TX_P
- IC1 pad 16: /Eth Switch/ETH3.TX_N -> /ETH3.TX_N
- J12 pad 10: (no net) -> GND
- J15 pad 21: /IO Connectors/ETH_DOCK.P0_P -> /ETH3.RX_P
- J15 pad 23: /IO Connectors/ETH_DOCK.P0_N -> /ETH3.RX_N
- J15 pad 25: /IO Connectors/ETH_DOCK.P1_P -> /ETH3.TX_P
- J15 pad 27: /IO Connectors/ETH_DOCK.P1_N -> /ETH3.TX_N
- J15 pad 3: /+5VPB -> /CM5/+3V3RPi
- J15 pad 6: /CM5/+3V3RPi -> /IO Connectors/PCTL_DBG_RST_N
- J15 pad 8: GND -> /IO Connectors/PCTL_DBG_BOOT
- SW2 pad 10: /CM5/WL_nDis -> unconnected-(SW2-Pad10)
- SW2 pad 11: /CM5/PWR_BUT -> /CM5/BT_nDis
- SW2 pad 12: /CM5/PMIC_ENABLE -> /CM5/WL_nDis
- SW2 pad 13: /CM5/USBOTG -> /CM5/PMIC_ENABLE
- SW2 pad 14: unconnected-(SW2-Pad14) -> /CM5/USBOTG
- SW2 pad 9: /CM5/BT_nDis -> unconnected-(SW2-Pad9)
- U7 pad 27: unconnected-(U7-GPA6-Pad27) -> Net-(J25-Pin_11)
- U7 pad 28: unconnected-(U7-GPA7-Pad28) -> Net-(J25-Pin_12)
- U7 pad 4: unconnected-(U7-GPB3-Pad4) -> Net-(J25-Pin_1)
- U7 pad 5: unconnected-(U7-GPB4-Pad5) -> Net-(J25-Pin_2)
- U7 pad 6: unconnected-(U7-GPB5-Pad6) -> Net-(J25-Pin_3)
- U7 pad 7: unconnected-(U7-GPB6-Pad7) -> Net-(J25-Pin_4)
- U7 pad 8: unconnected-(U7-GPB7-Pad8) -> Net-(J25-Pin_5)
Routing:
- net /CM5/MIPI1_ID_SCL: track 1.38 -> 97.2 mm, vias 1 -> 2
- net /CM5/MIPI1_ID_SDA: track 1.37 -> 96.2 mm, vias 1 -> 2
- net /CM5/USBC.CC2: track 0.00 -> 91.2 mm, vias 0 -> 2
- net /CM5/USBC.CC1: track 0.00 -> 88.9 mm, vias 0 -> 2
- net /Eth Switch/RMII.RXD0: track 0.00 -> 81.3 mm, vias 0 -> 1
- net /Eth Switch/RMII.CRS_DV: track 0.00 -> 80.1 mm, vias 0 -> 1
- net /Eth Switch/RMII.RXD1: track 0.00 -> 79.5 mm, vias 0 -> 1
- net /CM5/MIPI0_ID_SDA: track 0.66 -> 67.5 mm, vias 1 -> 2
- net /CM5/MIPI0_ID_SCL: track 0.53 -> 67.0 mm, vias 1 -> 2
- net /ETH3.RX_N: track 0.00 -> 62.2 mm, vias 0 -> 2
- net /CM5/CAM0_GPIO0: track 0.00 -> 61.8 mm, vias 0 -> 2
- net /Eth Switch/RMII.TXD1: track 0.00 -> 60.9 mm, vias 0 -> 1
- net /ETH3.RX_P: track 0.00 -> 60.0 mm, vias 0 -> 2
- net /CM5/CAM0_GPIO1: track 0.00 -> 58.9 mm, vias 0 -> 2
- net /Eth Switch/RMII.TXD0: track 0.00 -> 58.2 mm, vias 0 -> 1
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- added copper zone on In2.Cu, net /+VBUS_USBC
- removed copper zone on F.Cu, net /CM5/ETH.P1_P
Other:
- outline, holes or cut-outs redrawn
- board text added: "BOOT"
- board text added: "RST"
- board text added: "TODO: poprawić RMII"
