File: pcb_CMDB_Adv/Connectors.kicad_sch (KiCad schematic)
At the start: 22 parts, among them J11 CONN_SD, J12 CONN_USB3_A, J13 CONN_USB_PWR_OTG, J14 CONN_HAT, J15 CONN_DOCK, J16 CONN_CAM1, J17 CONN_CAM0, J6 CONN_UART3, J7 CONN_SPI, J8 CONN_I2C, J9 CONN_UART0, U6 AP22653W6

Commit message: CMDB-Adv PCB WIP
Parts:
- added J4: J_ESP_DBG_UART, Connector_Molex:Molex_PicoBlade_53047-0310_1x03_P1.25mm_Vertical, symbol Connector_Generic:Conn_01x03
- C19, C21, C22: Distributor TME -> (none); Part Description 10uF 10% 10V Ceramic Capacitor X7R -> (none)
- C20: Distributor TME -> (none); Part Description Capacitor, SP-Cap (Alu-Poly), 100u, 6.3V, 15mR ESR -> (none)
- J12: Distributor TME -> (none); Part Description USB 3.0 A connector -> (none)
- J13: Distributor TME -> (none); Part Description USBC USB2 data and power connector -> (none)
- J15: Distributor Mouser -> (none); Part Description High-Speed low raster 60-pin connector -> (none)
- J16, J17: Distributor Mouser -> (none); Part Description 22 Position FFC, FPC Connector Contacts, Bottom 0.020" (0.5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 -> (none)
- J6: value CONN_UART3 -> CONN_UART2; Field4 Farnell -> (none); Field5 1012259 -> (none); Field6 53048-0210 -> (none); Field7 Molex -> (none); Manufacturer (none) -> Molex; Part Description Pin Header, Right Angle, Signal, 1.25 mm, 1 Rows, 2 Contact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 -> (none); Part No. (none) -> 53048-0210
- J7: value CONN_SPI -> CONN_SPI1; Field4 Farnell -> (none); Field5 1012259 -> (none); Field6 53048-0210 -> (none); Field7 Molex -> (none); Manufacturer (none) -> Molex; Part Description Pin Header, Right Angle, Signal, 1.25 mm, 1 Rows, 2 Contact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 -> (none); Part No. (none) -> 53048-0210
- J8: value CONN_I2C -> CONN_I2C1; Field4 Farnell -> (none); Field5 1012259 -> (none); Field6 53048-0210 -> (none); Field7 Molex -> (none); Manufacturer (none) -> Molex; Part Description Pin Header, Right Angle, Signal, 1.25 mm, 1 Rows, 2 Contact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 -> (none); Part No. (none) -> 53048-0210
- J9: Field4 Farnell -> (none); Field5 1012259 -> (none); Field6 53048-0210 -> (none); Field7 Molex -> (none); Manufacturer (none) -> Molex; Part Description Pin Header, Right Angle, Signal, 1.25 mm, 1 Rows, 2 Contact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 -> (none); Part No. (none) -> 53048-0210
- R16, R18, R19, R20: Part Description Resistor 2.2K M1005 1% 63mW -> (none)
- R17: Part Description Resistor 15K M1005 1% 63mW -> (none)
- TP10: Distributor nf -> (none); Part Description Test point -> (none)
- U6: Distributor TME -> (none); Part Description Power Switch/Driver 1:1 P-Channel 2.1A SOT-23-6 -> (none)
Connections:
- net +3.3v_RPi is gone; now on net +3V3RPi: J14.1 (Pin_1), J14.17 (Pin_17)
- net +3.3v: no longer J15.4 (Pin_4), J16.22 (Pin_22), J17.22 (Pin_22), R18.2, R19.2, R20.1
- net +VBUS_USBA: now also J15.2 (Pin_2), J15.4 (Pin_4); no longer J15.5 (Pin_5), J15.7 (Pin_7)
- net GND: now also J15.8 (Pin_8), J4.1 (Pin_1); no longer J15.2 (Pin_2)
- net GP.4: now also J6.1 (Pin_1)
- net GP.5: now also J6.2 (Pin_2)
- net GP.8: no longer J6.1 (Pin_1)
- net GP.9: no longer J6.2 (Pin_2)
- net USB1.D_N: now also J12.2 (D-); no longer J12.6 (SSRX+)
- net USB1.D_P: now also J12.3 (D+); no longer J12.5 (SSRX-)
- net USB1.RX_N: now also J12.5 (SSRX-); no longer J12.2 (D-)
- net USB1.RX_P: now also J12.6 (SSRX+); no longer J12.3 (D+)
- net +3V3RPi: now reaches J15.6 (Pin_6)
- net +3V3RPi: now also J16.22 (Pin_22), J17.22 (Pin_22), R18.2, R19.2, R20.1
- net +5v renamed +5V
- net CC1 renamed USBC.CC1
- net CC2 renamed USBC.CC2
- net VBUS_EN renamed +VBUS_USBA_EN
- new net PCTL_DBG_UART_RX: J15.7 (Pin_7), J4.3 (Pin_3)
- new net PCTL_DBG_UART_TX: J15.5 (Pin_5), J4.2 (Pin_2)
Other:
- added sheet Ethernet Connectors (ethconn.kicad_sch)
- note added: "TODO: - Co z SD?"
- note added: "uart0 (14,15) routed uart1 (0,1) pins used for CAM (ID_SC/ID_SD) uart2 (4,5) routed uart3 (8,9) used for Platform Controller uart4 (12,13) pins unused uart10 - debug uart with CM5 header"
- note removed: "TODO: - FC UART - Other UARTs - GPIO solder-selectors (?) - I2Cs - I2C from ESP32 - LSHM: remove HDMI1? Add ESP prog lanes? Move USB-C to dock? - Co z SD?"
- moved on the sheet: C19, C20, C21, C22, J11, J15, R17, TP10, U6

Commit message: CMDB_Adv WIP
Parts:
- added TVS6: TPD4E1B06, symbol CMDB_Adv:TPD4E1B06
- J11: value CONN_SD -> CONN_SDIO; footprint (none) -> Connector_PinHeader_2.00mm:PinHeader_1x14_P2.00mm_Vertical
- J13: symbol Connector:USB_C_Receptacle_USB2.0_16P -> CMDB_Adv:USB_C_Receptacle_USB2.0_16P
Connections:
- net +3.3v is gone; now on net +3V3RPi: J11.1 (Pin_1)
- net +VBUS_USBA_EN is gone; now on net VBUS_USBA_EN: U6.3 (EN)
- net +VBUS_USBC: now also J13.A4_B9 (VBUS), J13.B4_A9 (VBUS); no longer J13.A4 (VBUS), J13.A9 (VBUS), J13.B4 (VBUS), J13.B9 (VBUS)
- net GND: now also J12.SH (SHIELD), J13.A1_B12 (GND), J13.B1_A12 (GND), J13.S2 (SHIELD), J13.S3 (SHIELD), J13.S4 (SHIELD); no longer J12.10 (SHIELD), J13.A1 (GND), J13.A12 (GND), J13.B1 (GND), J13.B12 (GND)
- net ETH1.P0_N renamed ETH_DOCK.P0_N
- net ETH1.P0_P renamed ETH_DOCK.P0_P
- net ETH1.P1_N renamed ETH_DOCK.P1_N
- net ETH1.P1_P renamed ETH_DOCK.P1_P
- net ETH1.P2_N renamed ETH_DOCK.P2_N
- net ETH1.P2_P renamed ETH_DOCK.P2_P
- net ETH1.P3_N renamed ETH_DOCK.P3_N
- net ETH1.P3_P renamed ETH_DOCK.P3_P
- new net: TVS6.1 (IO1), TVS6.10
- new net: TVS6.2 (IO2), TVS6.9
- new net: TVS6.3 (GND), TVS6.8 (GND)
- new net: TVS6.4 (IO3), TVS6.7
- new net: TVS6.5 (IO4), TVS6.6
Other:
- note added: "I2C1_SCL"
- note added: "I2C1_SDA"
- note added: "SPI1_CS0"
- note added: "SPI1_CS1"
- note added: "SPI1_MISO"
- note added: "SPI1_MOSI"
- note added: "SPI1_SCLK"
- note added: "TODO: - Co z SD? - TVS na oba USB"
- note added: "UART0_RX"
- note added: "UART0_TX"
- note added: "UART2_RX"
- note added: "UART2_TX"
- note removed: "TODO: - Co z SD?"

Commit message: WIP
Other:
- moved on the sheet: TVS6
Changed lines of the file:
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@@
 	(rectangle
 		(start 149.86 15.24)
-		(end 232.41 82.55)
+		(end 232.41 95.25)
 		(stroke
 			(width 0)
@@
 	(text "uart0 (14,15) routed\nuart1 (0,1) pins used for CAM (ID_SC/ID_SD)\nuart2 (4,5) routed\nuart3 (8,9) used for Platform Controller\nuart4 (12,13) pins unused\nuart10 - debug uart with CM5 header\n"
 		(exclude_from_sim no)
-		(at 191.008 88.9 0)
+		(at 198.882 88.646 0)
 		(effects
 			(font
@@
 	(text "TODO:\n- Co z SD?\n- TVS na oba USB"
 		(exclude_from_sim no)
-		(at 26.924 96.52 0)
+		(at 34.544 95.25 0)
 		(effects
 			(font
@@
 	(symbol
 		(lib_id "CMDB_Adv:TPD4E1B06")
-		(at 15.24 100.33 90)
+		(at 22.86 99.06 90)
 		(mirror x)
 		(unit 1)
@@
 		(dnp no)
 		(property "Reference" "TVS6"
-			(at 15.24 107.696 90)
+			(at 22.86 106.426 90)
 			(show_name no)
 			(do_not_autoplace no)
@@
 		)
 		(property "Value" "TPD4E1B06"
-			(at 15.24 100.33 0)
+			(at 22.86 99.06 0)
 			(show_name no)
 			(do_not_autoplace no)
@@
 		)
 		(property "Footprint" ""
-			(at 15.24 100.33 0)
+			(at 22.86 99.06 0)
 			(hide yes)
 			(show_name no)
@@
 		)
 		(property "Datasheet" ""
-			(at 15.24 100.33 0)
+			(at 22.86 99.06 0)
 			(hide yes)
 			(show_name no)
@@
 		)
 		(property "Description" ""
-			(at 15.24 100.33 0)
+			(at 22.86 99.06 0)
 			(hide yes)
 			(show_name no)

Commit message: WIP CMDB-Adv
Connections:
- net +3V3RPi: now also J15.3 (Pin_3); no longer J15.6 (Pin_6)
- net +5V: no longer J15.3 (Pin_3)
- net GND: now also J12.10 (SHIELD); no longer J12.SH (SHIELD), J15.8 (Pin_8)
- new net PCTL_DBG_BOOT: J15.8 (Pin_8)
- new net PCTL_DBG_RST_N: J15.6 (Pin_6)
Other:
- note added: "TODO: - TVS na oba USB"
- note removed: "TODO: - Co z SD? - TVS na oba USB"
- moved on the sheet: TVS6
Changed lines of the file:
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@@
 		)
 	)
-	(text "TODO:\n- Co z SD?\n- TVS na oba USB"
+	(text "TODO:\n- TVS na oba USB"
 		(exclude_from_sim no)
-		(at 34.544 95.25 0)
+		(at 5.334 97.79 0)
 		(effects
 			(font
@@
 	)
 	(junction
-		(at 113.03 31.75)
-		(diameter 0)
-		(color 0 0 0 0)
-	)
-	(junction
 		(at 97.79 90.17)
 		(diameter 0)
@@
 	(bus
 		(pts
-			(xy 33.02 62.23) (xy 52.07 62.23)
+			(xy 33.02 66.04) (xy 52.07 66.04)
 		)
 		(stroke
@@
 	(wire
 		(pts
+			(xy 127 29.21) (xy 111.76 29.21)
+		)
+		(stroke
+			(width 0)
+			(type default)
+		)
+	)
+	(wire
+		(pts
 			(xy 218.44 25.4) (xy 227.33 25.4)
 		)
@@
 	(bus
 		(pts
-			(xy 33.02 64.77) (xy 52.07 64.77)
+			(xy 33.02 68.58) (xy 52.07 68.58)
 		)
 		(stroke
@@
 	(bus
 		(pts
-			(xy 33.02 78.74) (xy 52.07 78.74)
+			(xy 33.02 82.55) (xy 52.07 82.55)
 		)
 		(stroke
@@
 		)
 	)
+	(wire
+		(pts
+			(xy 33.02 58.42) (xy 52.07 58.42)
+		)
+		(stroke
+			(width 0)
+			(type default)
+		)
+	)
 	(bus
 		(pts
@@
 	(bus
 		(pts
-			(xy 33.02 85.09) (xy 52.07 85.09)
+			(xy 33.02 88.9) (xy 52.07 88.9)
 		)
 		(stroke
@@
 	(bus
 		(pts
-			(xy 33.02 76.2) (xy 52.07 76.2)
+			(xy 33.02 80.01) (xy 52.07 80.01)
 		)
 		(stroke
@@
 	(wire
 		(pts
+			(xy 127 26.67) (xy 111.76 26.67)
+		)
+		(stroke
+			(width 0)
+			(type default)
+		)
+	)
+	(wire
+		(pts
 			(xy 97.79 74.93) (xy 97.79 82.55)
 		)
@@
 		)
 	)
+	(wire
+		(pts
+			(xy 33.02 60.96) (xy 52.07 60.96)
+		)
+		(stroke
+			(width 0)
+			(type default)
+		)
+	)
 	(polyline
 		(pts
@@
 	(bus
 		(pts
-			(xy 33.02 82.55) (xy 52.07 82.55)
+			(xy 33.02 86.36) (xy 52.07 86.36)
 		)
 		(stroke
@@
 	(wire
 		(pts
-			(xy 113.03 29.21) (xy 113.03 31.75)
-		)
-		(stroke
-			(width 0)
-			(type default)
-		)
-	)
-	(wire
-		(pts
 			(xy 226.06 154.94) (xy 222.25 154.94)
 		)
@@
 	(bus
 		(pts
-			(xy 33.02 68.58) (xy 52.07 68.58)
+			(xy 33.02 72.39) (xy 52.07 72.39)
 		)
 		(stroke
@@
 	(bus
 		(pts
-			(xy 33.02 71.12) (xy 52.07 71.12)
+			(xy 33.02 74.93) (xy 52.07 74.93)
 		)
 		(stroke
@@
 		)
 	)
-	(wire
-		(pts
-			(xy 111.76 29.21) (xy 113.03 29.21)
-		)
-		(stroke
-			(width 0)
-			(type default)
-		)
-	)
 	(polyline
 		(pts
@@
 	(wire
 		(pts
-			(xy 124.46 26.67) (xy 111.76 26.67)
-		)
-		(stroke
-			(width 0)
-			(type default)
-		)
-	)
-	(wire
-		(pts
 			(xy 158.75 41.91) (xy 181.61 41.91)
 		)
@@
 	)
 	(label "MIPI1{MIPI}"
-		(at 52.07 85.09 180)
+		(at 52.07 88.9 180)
 		(effects
 			(font
@@
 	)
 	(label "MIPI0{MIPI}"
-		(at 52.07 82.55 180)
+		(at 52.07 86.36 180)
 		(effects
 			(font
@@
 	)
 	(label "HDMI0{HDMI}"
-		(at 52.07 68.58 180)
+		(at 52.07 72.39 180)
 		(effects
 			(font
@@
 		)
 	)
-	(label "+5V"
-		(at 86.36 24.13 0)
-		(effects
-			(font
-				(size 1.27 1.27)
-			)
-			(justify left bottom)
-		)
-	)
 	(label "HDMI0.SCL"
 		(at 86.36 34.29 0)
@@
 	)
 	(label "HDMI1{HDMI}"
-		(at 52.07 71.12 180)
+		(at 52.07 74.93 180)
 		(effects
 			(font
@@
 	)
 	(label "SD{SD}"
-		(at 52.07 64.77 180)
+		(at 52.07 68.58 180)
 		(effects
 			(font
@@
 		)
 	)
+	(label "PCTL_DBG_BOOT"
+		(at 52.07 60.96 180)
+		(effects
+			(font
+				(size 1.27 1.27)
+			)
+			(justify right bottom)
+		)
+	)
 	(label "SD.DAT4"
 		(at 166.37 115.57 180)
@@
 		)
 	)
-	(label "HDMI1.HP"
-		(at 124.46 41.91 180)
+	(label "PCTL_DBG_RST_N"
+		(at 52.07 58.42 180)
 		(effects
 			(font
@@
 		)
 	)
-	(label "VBUS_USBA_EN"
-		(at 52.07 31.75 180)
+	(label "HDMI1.HP"
+		(at 124.46 41.91 180)
 		(effects
 			(font
@@
 		)
 	)
-	(label "+3V3RPi"
-		(at 124.46 26.67 180)
+	(label "VBUS_USBA_EN"
+		(at 52.07 31.75 180)
 		(effects
 			(font
@@
 		)
 	)
+	(label "PCTL_DBG_RST_N"
+		(at 127 26.67 180)
+		(effects
+			(font
+				(size 1.27 1.27)
+			)
+			(justify right bottom)
+		)
+	)
 	(label "+3V3RPi"
 		(at 69.85 116.84 0)
@@
 	)
 	(label "USB0{USB}"
-		(at 52.07 76.2 180)
+		(at 52.07 80.01 180)
 		(effects
 			(font
@@
 	)
 	(label "USBC{USBC}"
-		(at 52.07 62.23 180)
+		(at 52.07 66.04 180)
 		(effects
 			(font
@@
 	)
 	(label "USB1{USB}"
-		(at 52.07 78.74 180)
+		(at 52.07 82.55 180)
 		(effects
 			(font
@@
 		)
 	)
+	(label "+3V3RPi"
+		(at 86.36 24.13 0)
+		(effects
+			(font
+				(size 1.27 1.27)
+			)
+			(justify left bottom)
+		)
+	)
 	(label "MIPI0.D1_N"
 		(at 254 35.56 0)
@@
 		)
 	)
+	(label "PCTL_DBG_BOOT"
+		(at 127 29.21 180)
+		(effects
+			(font
+				(size 1.27 1.27)
+			)
+			(justify right bottom)
+		)
+	)
 	(label "USB0.TX_P"
 		(at 124.46 64.77 180)
@@
 		)
 	)
+	(hierarchical_label "PCTL_DBG_BOOT"
+		(shape input)
+		(at 33.02 60.96 180)
+		(effects
+			(font
+				(size 1.27 1.27)
+			)
+			(justify right)
+		)
+	)
 	(hierarchical_label "MIPI0_ID_SDA"
 		(shape bidirectional)
@@
 	(hierarchical_label "HDMI0{HDMI}"
 		(shape input)
-		(at 33.02 68.58 180)
+		(at 33.02 72.39 180)
+		(effects
+			(font
+				(size 1.27 1.27)
+			)
+			(justify right)
+		)
+	)
+	(hierarchical_label "PCTL_DBG_RST_N"
+		(shape input)
+		(at 33.02 58.42 180)
 		(effects
 			(font
@@
 	(hierarchical_label "USBC{USBC}"
 		(shape bidirectional)
-		(at 33.02 62.23 180)
+		(at 33.02 66.04 180)
 		(effects
 			(font
@@
 	(hierarchical_label "HDMI1{HDMI}"
 		(shape input)
-		(at 33.02 71.12 180)
+		(at 33.02 74.93 180)
 		(effects
 			(font
@@
 	(hierarchical_label "USB0{USB}"
 		(shape bidirectional)
-		(at 33.02 76.2 180)
+		(at 33.02 80.01 180)
 		(effects
 			(font
@@
 	(hierarchical_label "SD{SD}"
 		(shape bidirectional)
-		(at 33.02 64.77 180)
+		(at 33.02 68.58 180)
 		(effects
 			(font
@@
 	(hierarchical_label "USB1{USB}"
 		(shape bidirectional)
-		(at 33.02 78.74 180)
+		(at 33.02 82.55 180)
 		(effects
 			(font
@@
 	(hierarchical_label "MIPI1{MIPI}"
 		(shape bidirectional)
-		(at 33.02 85.09 180)
+		(at 33.02 88.9 180)
 		(effects
 			(font
@@
 	(hierarchical_label "MIPI0{MIPI}"
 		(shape bidirectional)
-		(at 33.02 82.55 180)
+		(at 33.02 86.36 180)
 		(effects
 			(font
@@
 	(symbol
 		(lib_id "CMDB_Adv:TPD4E1B06")
-		(at 22.86 99.06 90)
+		(at -6.35 101.6 90)
 		(mirror x)
 		(unit 1)
@@
 		(dnp no)
 		(property "Reference" "TVS6"
-			(at 22.86 106.426 90)
+			(at -6.35 110.998 90)
 			(show_name no)
 			(do_not_autoplace no)
@@
 		)
 		(property "Value" "TPD4E1B06"
-			(at 22.86 99.06 0)
+			(at -6.35 108.712 90)
 			(show_name no)
 			(do_not_autoplace no)
@@
 		)
 		(property "Footprint" ""
-			(at 22.86 99.06 0)
+			(at -6.35 101.6 0)
 			(hide yes)
 			(show_name no)
@@
 		)
 		(property "Datasheet" ""
-			(at 22.86 99.06 0)
+			(at -6.35 101.6 0)
 			(hide yes)
 			(show_name no)
@@
 		)
 		(property "Description" ""
-			(at 22.86 99.06 0)
+			(at -6.35 101.6 0)
 			(hide yes)
 			(show_name no)
@@
 			)
 		)
-		(pin "SH"
+		(pin "10"
 		)
 		(pin "7"
