File: pcb_CMDB_Adv/PCIe-M2.kicad_sch (KiCad schematic)
At the start: 11 parts, among them J2 Bus_M.2_Socket_M, M1 M.2 Solder Nut, M2 M.2 Solder Nut, M3 M.2 Screw, U1 ASEK-32.768KHZ-L-R-T

Commit message: CMDB-Adv PCB WIP
Parts:
- C1, C2: Distributor TME -> (none); Part Description 10uF 10% 10V Ceramic Capacitor X7R -> (none)
- C3: Distributor TME -> (none); Part Description 0.1uF 10% 16V Ceramic Capacitor X7R -> (none)
- D1: Distributor Mouser -> (none); Part Description Green 572nm LED Indication - Discrete 2.2V 2-SMD, No Lead -> (none)
- J2: Part Description M.2 Socket 3 Mechanical Key M -> (none)
- M1, M2: Part Description Solder nut for M.2 slot -> (none)
- M3: Part Description M.2 Screw -> (none)
- R1: Part Description Resistor 1K M1005 1% 63mW -> (none)
- TP1: Distributor nf -> (none); Part Description Test point -> (none)
- U1: Part Description 32KHz Xtal oscilator -> (none)
Connections:
- net PCIe.RX_N renamed DEVICE_RX_N
- net PCIe.RX_P renamed DEVICE_RX_P
- net PCIe.TX_N renamed DEVICE_TX_N
- net PCIe.TX_P renamed DEVICE_TX_P

Commit message: CMDB_Adv WIP
Parts:
- removed C1, C2: 10u, Capacitor_SMD:C_0805_2012Metric_Pad1.18x1.45mm_HandSolder, symbol Device:C
- removed TP1: TestPoint, TestPoint:TestPoint_Pad_2.0x2.0mm, symbol Connector:TestPoint
- added C58, C72, C73: 22uF, Capacitor_SMD:C_1206_3216Metric_Pad1.33x1.80mm_HandSolder, symbol Device:C
- added D3: LED Red, LED_SMD:LED_0603_1608Metric, symbol Device:LED
- added R2: 1K, Resistor_SMD:R_0805_2012Metric_Pad1.20x1.40mm_HandSolder, symbol Device:R
- J2: footprint CMDB_Adv:M.2 M Key socket -> CMDB_Adv:M.2_M_Key_socket_2280; symbol CM5IO:Bus_M.2_Socket_M -> CMDB_Adv:Bus_M.2_Socket_M
- M1, M2: symbol CM5IO:SolderNut -> CMDB_Adv:SolderNut
- M3: symbol CM5IO:M.2_Screw -> CMDB_Adv:M.2_Screw
- U1: symbol CM5IO:ASEK-32.768KHZ-L-R-T -> CMDB_Adv:ASEK-32.768KHZ-L-R-T
Connections:
- net M2_3V3 is gone; now on net +3V3_M2: D1.2 (A), J2.12 (3.3V), J2.14 (3.3V), J2.16 (3.3V), J2.18 (3.3V), J2.2 (3.3V), J2.4 (3.3V), J2.70 (3.3V), J2.72 (3.3V), J2.74 (3.3V), U1.1 (EN)
- net GND: now also C58.1, C72.1, C73.1, R2.2
- net +3.3v_M2 renamed +3V3_M2
- net +3V3_M2: now also C58.2, C72.2, C73.2, D3.2 (A)
- net DEVICE_RX_N renamed PCIe.RX_N
- net DEVICE_RX_P renamed PCIe.RX_P
- net DEVICE_TX_N renamed PCIe.TX_N
- net DEVICE_TX_P renamed PCIe.TX_P
- new net: D3.1 (K), R2.1
Other:
- note added: "DEVICE_RX_N"
- note added: "DEVICE_RX_P"
- note added: "DEVICE_TX_N"
- note added: "DEVICE_TX_P"
- note added: "PCIe PWR LED"
- moved on the sheet: D1

Commit message: WIP
Parts:
- added M4, M5: M.2 Solder Nut, symbol CMDB_Adv:SolderNut
Other:
- moved on the sheet: M1, M2, M3
Changed lines of the file:
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@@
+	)
+	(symbol
+		(lib_id "CMDB_Adv:SolderNut")
+		(at 276.86 143.51 0)
+		(mirror y)
+		(unit 1)
+		(body_style 1)
+		(exclude_from_sim yes)
+		(in_bom yes)
+		(on_board no)
+		(in_pos_files yes)
+		(dnp no)
+		(fields_autoplaced yes)
+		(property "Reference" "M5"
+			(at 271.78 142.2399 0)
+			(show_name no)
+			(do_not_autoplace no)
+			(effects
+				(font
+					(size 1.27 1.27)
+				)
+				(justify left)
+			)
+		)
+		(property "Value" "M.2 Solder Nut"
+			(at 271.78 144.7799 0)
+			(show_name no)
+			(do_not_autoplace no)
+			(effects
+				(font
+					(size 1.27 1.27)
+				)
+				(justify left)
+			)
+		)
+		(property "Footprint" ""
+			(at 276.86 143.51 0)
+			(hide yes)
+			(show_name no)
+			(do_not_autoplace no)
+			(effects
+				(font
+					(size 1.27 1.27)
+				)
+			)
+		)
+		(property "Datasheet" ""
+			(at 276.86 143.51 0)
+			(hide yes)
+			(show_name no)
+			(do_not_autoplace no)
+			(effects
+				(font
+					(size 1.27 1.27)
+				)
+			)
+		)
+		(property "Description" "Solder nut for M.2 slot"
+			(at 276.86 143.51 0)
+			(hide yes)
+			(show_name no)
+			(do_not_autoplace no)
+			(effects
+				(font
+					(size 1.27 1.27)
+				)
+			)
+		)
+		(instances
+			(project "CMDB_Adv"
+				(path "/e63e39d7-6ac0-4ffd-8aa3-1841a4541b55/bcd581d4-623c-482f-9f93-14cd226a9d2f"
+					(reference "M5")
+					(unit 1)
+				)
+			)
+		)
+	)
+	(symbol
+		(lib_id "CMDB_Adv:SolderNut")
+		(at 276.86 133.35 0)
+		(mirror y)
+		(unit 1)
+		(body_style 1)
+		(exclude_from_sim yes)
+		(in_bom yes)
+		(on_board no)
+		(in_pos_files yes)
+		(dnp no)
+		(fields_autoplaced yes)
+		(property "Reference" "M4"
+			(at 271.78 132.0799 0)
+			(show_name no)
+			(do_not_autoplace no)
+			(effects
+				(font
+					(size 1.27 1.27)
+				)
+				(justify left)
+			)
+		)
+		(property "Value" "M.2 Solder Nut"
+			(at 271.78 134.6199 0)
+			(show_name no)
+			(do_not_autoplace no)
+			(effects
+				(font
+					(size 1.27 1.27)
+				)
+				(justify left)
+			)
+		)
+		(property "Footprint" ""
+			(at 276.86 133.35 0)
+			(hide yes)
+			(show_name no)
+			(do_not_autoplace no)
+			(effects
+				(font
+					(size 1.27 1.27)
+				)
+			)
+		)
+		(property "Datasheet" ""
+			(at 276.86 133.35 0)
+			(hide yes)
+			(show_name no)
+			(do_not_autoplace no)
+			(effects
+				(font
+					(size 1.27 1.27)
+				)
+			)
+		)
+		(property "Description" "Solder nut for M.2 slot"
+			(at 276.86 133.35 0)
+			(hide yes)
+			(show_name no)
+			(do_not_autoplace no)
+			(effects
+				(font
+					(size 1.27 1.27)
+				)
+			)
+		)
+		(instances
+			(project "CMDB_Adv"
+				(path "/e63e39d7-6ac0-4ffd-8aa3-1841a4541b55/bcd581d4-623c-482f-9f93-14cd226a9d2f"
+					(reference "M4")
+					(unit 1)
+				)
+			)
+		)
 	)
 	(symbol
 		(lib_id "CMDB_Adv:M.2_Screw")
-		(at 260.35 142.24 0)
+		(at 275.59 157.48 0)
+		(mirror y)
 		(unit 1)
 		(body_style 1)
@@
 		(fields_autoplaced yes)
 		(property "Reference" "M3"
-			(at 267.97 140.9699 0)
+			(at 267.97 156.2099 0)
 			(show_name no)
 			(do_not_autoplace no)
@@
 		)
 		(property "Value" "M.2 Screw"
-			(at 267.97 143.5099 0)
+			(at 267.97 158.7499 0)
 			(show_name no)
 			(do_not_autoplace no)
@@
 		)
 		(property "Footprint" ""
-			(at 260.35 142.24 0)
-			(hide yes)
-			(show_name no)
-			(do_not_autoplace no)
-			(effects
-				(font
-					(size 1.27 1.27)
-				)
-			)
-		)
-		(property "Datasheet" ""
-			(at 260.35 142.24 0)
+			(at 275.59 157.48 0)
+			(hide yes)
+			(show_name no)
+			(do_not_autoplace no)
+			(effects
+				(font
+					(size 1.27 1.27)
+				)
+			)
+		)
+		(property "Datasheet" ""
+			(at 275.59 157.48 0)
 			(hide yes)
 			(show_name no)
@@
 		)
 		(property "Description" "M.2 Screw"
-			(at 260.35 142.24 0)
+			(at 275.59 157.48 0)
 			(hide yes)
 			(show_name no)
@@
 	(symbol
 		(lib_id "CMDB_Adv:SolderNut")
-		(at 257.81 125.73 0)
+		(at 276.86 123.19 0)
+		(mirror y)
 		(unit 1)
 		(body_style 1)
@@
 		(fields_autoplaced yes)
 		(property "Reference" "M2"
-			(at 262.89 124.4599 0)
+			(at 271.78 121.9199 0)
 			(show_name no)
 			(do_not_autoplace no)
@@
 		)
 		(property "Value" "M.2 Solder Nut"
-			(at 262.89 126.9999 0)
+			(at 271.78 124.4599 0)
 			(show_name no)
 			(do_not_autoplace no)
@@
 		)
 		(property "Footprint" ""
-			(at 257.81 125.73 0)
-			(hide yes)
-			(show_name no)
-			(do_not_autoplace no)
-			(effects
-				(font
-					(size 1.27 1.27)
-				)
-			)
-		)
-		(property "Datasheet" ""
-			(at 257.81 125.73 0)
+			(at 276.86 123.19 0)
+			(hide yes)
+			(show_name no)
+			(do_not_autoplace no)
+			(effects
+				(font
+					(size 1.27 1.27)
+				)
+			)
+		)
+		(property "Datasheet" ""
+			(at 276.86 123.19 0)
 			(hide yes)
 			(show_name no)
@@
 		)
 		(property "Description" "Solder nut for M.2 slot"
-			(at 257.81 125.73 0)
+			(at 276.86 123.19 0)
 			(hide yes)
 			(show_name no)
@@
 	(symbol
 		(lib_id "CMDB_Adv:SolderNut")
-		(at 257.81 113.03 0)
+		(at 276.86 113.03 0)
+		(mirror y)
 		(unit 1)
 		(body_style 1)
@@
 		(fields_autoplaced yes)
 		(property "Reference" "M1"
-			(at 262.89 111.7599 0)
+			(at 271.78 111.7599 0)
 			(show_name no)
 			(do_not_autoplace no)
@@
 		)
 		(property "Value" "M.2 Solder Nut"
-			(at 262.89 114.2999 0)
+			(at 271.78 114.2999 0)
 			(show_name no)
 			(do_not_autoplace no)
@@
 		)
 		(property "Footprint" ""
-			(at 257.81 113.03 0)
-			(hide yes)
-			(show_name no)
-			(do_not_autoplace no)
-			(effects
-				(font
-					(size 1.27 1.27)
-				)
-			)
-		)
-		(property "Datasheet" ""
-			(at 257.81 113.03 0)
+			(at 276.86 113.03 0)
+			(hide yes)
+			(show_name no)
+			(do_not_autoplace no)
+			(effects
+				(font
+					(size 1.27 1.27)
+				)
+			)
+		)
+		(property "Datasheet" ""
+			(at 276.86 113.03 0)
 			(hide yes)
 			(show_name no)
@@
 		)
 		(property "Description" "Solder nut for M.2 slot"
-			(at 257.81 113.03 0)
-			(hide yes)
-			(show_name no)
+			(at 276.86 113.03 0)
+			(hide yes)
+			(show_name no)

Commit message: WIP CMDB-Adv
Parts:
- M1, M2, M3, M4, M5: now not fitted
Changed lines of the file:
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@@
 		(on_board no)
 		(in_pos_files yes)
-		(dnp no)
+		(dnp yes)
 		(fields_autoplaced yes)
 		(property "Reference" "M5"
@@
 		(on_board no)
 		(in_pos_files yes)
-		(dnp no)
+		(dnp yes)
 		(fields_autoplaced yes)
 		(property "Reference" "M4"
@@
 		(on_board no)
 		(in_pos_files yes)
-		(dnp no)
+		(dnp yes)
 		(fields_autoplaced yes)
 		(property "Reference" "M3"
@@
 		(on_board no)
 		(in_pos_files yes)
-		(dnp no)
+		(dnp yes)
 		(fields_autoplaced yes)
 		(property "Reference" "M2"
@@
 		(on_board no)
 		(in_pos_files yes)
-		(dnp no)
+		(dnp yes)
 		(fields_autoplaced yes)
 		(property "Reference" "M1"
