File: pcb_CMDB_Adv/PlCtrl.kicad_sch (KiCad schematic)
At the start: 25 parts, among them IC2 Wio-SX1262, J4 J_ESP_DBG_UART, SW3 SW_RESET, SW4 SW_BOOT, U5 ESP32-WROOM-32UE, U7 MCP23017_SO

Commit message: CMDB-Adv PCB WIP
Parts:
- removed C10: 10uF, Capacitor_SMD:C_0805_2012Metric_Pad1.18x1.45mm_HandSolder, symbol Device:C_Small
- removed C15, C16: 470nF, Capacitor_SMD:C_0805_2012Metric_Pad1.18x1.45mm_HandSolder, symbol Device:C_Small
- removed J4: J_ESP_DBG_UART, Connector_Molex:Molex_PicoBlade_53047-0310_1x03_P1.25mm_Vertical, symbol Connector_Generic:Conn_01x03
- added C41: 10uF, Capacitor_SMD:C_1206_3216Metric_Pad1.33x1.80mm_HandSolder, symbol Device:C_Small
- added C43, C49: 22uF, Capacitor_SMD:C_1206_3216Metric_Pad1.33x1.80mm_HandSolder, symbol Device:C
- added C44, C50, C51, C52: 100nF, Capacitor_SMD:C_0402_2012Metric_Pad1.18x1.45mm_HandSolder, symbol Device:C_Small
- D8: Field4 Digikey -> (none); Field5 LTST-S270KGKT -> (none); Field6 SML-A12M8TT86N -> (none); Field7 Rohm -> (none); Field8 650263301 -> (none); Manufacturer (none) -> LITEON; Part Description Green 572nm LED Indication - Discrete 2.2V 2-SMD, No Lead -> (none); Part No. (none) -> LTST-S270KGKT
- IC2: footprint 114993390 -> CMDB_Adv:Wio-SX1262; Height 3.15 -> (none); Manufacturer_Name Seeed Studio -> (none); Manufacturer_Part_Number 114993390 -> (none); Mouser Part Number 713-114993390 -> (none); Mouser Price/Stock https://www.mouser.co.uk/ProductDetail/Seeed-Studio/1149933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 -> (none)
- SW3, SW4: Field4 Farnell -> (none); Field5 1201424 -> (none); Field6 KMR221G LFS -> (none); Field7 C&K COMPONENTS -> (none); Manufacturer (none) -> C&K COMPONENTS; Part Description Tactile Switch, KMR 2 Series, Top Actuated, Surface Mount, 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 -> (none); Part No. (none) -> KMR221G LFS
- U5: Part No. (none) -> ESP32-WROOM-32UE
- U7: Part No. (none) -> MCP23017
Connections:
- net +3.3v_LoRa is gone; now on net +3V3_LoRa: IC2.8 (VCC)
- net +3.3v_ESP: no longer R13.1
- net +3V3_ESP: now also R13.1, C49.2, C50.2, C51.2, C52.2
- net +3V3_LoRa: now also C43.2, C44.2
- net GND: now also C41.2, C43.1, C44.1, C49.1, C50.1, C51.1, C52.1
- net SWITCH_RST_N: now also C41.1
- net UART_RX: no longer U5.4 (SENSOR_VP)
- net UART_TX: no longer U5.23 (IO15)
- net +5VPB_EN: now reaches U7.21 (GPA0)
- net +5VEXT1_EN: now reaches U7.22 (GPA1)
- net +5VEXT2_EN: now reaches U7.23 (GPA2)
- new net RPi_UART_RX: U5.4 (SENSOR_VP)
- new net RPi_UART_TX: U5.23 (IO15)
Other:
- note added: "SWITCH MISC"
- note added: "TODO: Platform Controller IO TODO: Killswitch!!!"
- note removed: "TODO: RPi UART!!!"
- moved on the sheet: C8, D8, D9, IC2, JP10, JP6, JP7, JP8, JP9, R13, R14, R15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

Commit message: CMDB_Adv WIP
Parts:
- removed C41: 10uF, Capacitor_SMD:C_1206_3216Metric_Pad1.33x1.80mm_HandSolder, symbol Device:C_Small
- removed D9: 1N4148, symbol Device:D_Small_Filled
- removed R23: 10K, Resistor_SMD:R_0805_2012Metric_Pad1.20x1.40mm_HandSolder, symbol Device:R_Small
- added C53: 10uF, Capacitor_SMD:C_1206_3216Metric_Pad1.33x1.80mm_HandSolder, symbol Device:C_Small
- added D15: BAT54A, Package_TO_SOT_SMD:SOT-23, symbol Diode:BAT54A
- added R44: 10K, Resistor_SMD:R_0805_2012Metric_Pad1.20x1.40mm_HandSolder, symbol Device:R_Small
- added R52, R53, R54, R55, R56, R57: 22R, Resistor_SMD:R_0805_2012Metric_Pad1.20x1.40mm_HandSolder, symbol Device:R_Small
- C44, C50, C51, C52: footprint Capacitor_SMD:C_0402_2012Metric_Pad1.18x1.45mm_HandSolder -> Capacitor_SMD:C_0402_1005Metric_Pad0.74x0.62mm_HandSolder
- U7: symbol Interface_Expansion:MCP23017_SO -> Interface_Expansion:MCP23017x-x-SO
Connections:
- net +3.3v_ESP is gone; now on net +3V3_ESP: R14.1, R15.1
- net +3V3_ESP: now also D15.1, R44.2
- net +5VEXT1_EN: now also U7.2 (GPB1); no longer U7.22 (GPA1)
- net +5VEXT2_EN: now also U7.3 (GPB2); no longer U7.23 (GPA2)
- net +5VPB_EN: now also U7.1 (GPB0); no longer U7.21 (GPA0)
- net ADDR1: now also U7.21 (GPA0); no longer U7.1 (GPB0)
- net ADDR16: now also U7.25 (GPA4); no longer U7.5 (GPB4)
- net ADDR2: now also U7.22 (GPA1); no longer U7.2 (GPB1)
- net ADDR4: now also U7.23 (GPA2); no longer U7.3 (GPB2)
- net ADDR8: now also U7.24 (GPA3); no longer U7.4 (GPB3)
- net ENABLE: now also D15.2
- net GND: now also U5.[1,15,38,39] (GND), C53.2; no longer U5.1 (GND), U5.15 (GND), U5.38 (GND), U5.39 (GND)
- net LED_ACT: now also U7.26 (GPA5); no longer U7.6 (GPB5)
- net RMII.CRS_DV: now also R57.1; no longer U5.12 (IO27)
- net RMII.RXD0: now also R55.1; no longer U5.10 (IO25)
- net RMII.RXD1: now also R56.1; no longer U5.11 (IO26)
- net RMII.TXD0: now also R52.1; no longer U5.31 (IO19)
- net RMII.TXD1: now also R54.1; no longer U5.36 (IO22)
- net RMII.TX_EN: now also R53.1; no longer U5.33 (IO21)
- net SWITCH_RST_N: now also C53.1, D15.3, R44.1
- net SWITCH_INT: now reaches U5.5 (SENSOR_VN)
- net LORA.CS renamed LORA_CS
- net LORA.MISO renamed SPI.MISO
- net LORA.MOSI renamed SPI.MOSI
- net LORA.SCLK renamed SPI.SCLK
- net SWITCH.CS renamed SPI.CS
- new net: R55.2, U5.10 (IO25)
- new net: R57.2, U5.12 (IO27)
- new net: R53.2, U5.33 (IO21)
- new net: R56.2, U5.11 (IO26)
- new net: R52.2, U5.31 (IO19)
- new net: R54.2, U5.36 (IO22)
- no-connect marks 5 -> 12
Other:
- note added: "ETHERNET SWITCH MISC"
- note added: "KSZ8795 reset sequencing Holds RST_N low ~100 ms after ESP32 boot. (Delayed start to avoid feeding IO0 with clock before ESP32 boots up.) IO4 should be in high-z before boot."
- note removed: "Delayed start circuit for switch to avoid feeding IO0 with clock before ESP32 boots up. IO4 should be in high-z before boot."
- note removed: "SWITCH MISC"
- moved on the sheet: JP10, JP6, JP7, JP8, JP9, R13, R22, U5

Commit message: WIP
Parts:
- added J25: PL_CTRL_IO, symbol Connector_Generic:Conn_02x06_Counter_Clockwise
Connections:
- net +3V3_ESP: now also J25.8 (Pin_8)
- net GND: now also J25.6 (Pin_6), J25.7 (Pin_7)
- net I2C_SCL: now also J25.9 (Pin_9)
- net I2C_SDA: now also J25.10 (Pin_10)
- net at U7.27 (GPA6): now also J25.11 (Pin_11)
- net at U7.28 (GPA7): now also J25.12 (Pin_12)
- net at U7.4 (GPB3): now also J25.1 (Pin_1)
- net at U7.5 (GPB4): now also J25.2 (Pin_2)
- net at U7.6 (GPB5): now also J25.3 (Pin_3)
- net at U7.7 (GPB6): now also J25.4 (Pin_4)
- net at U7.8 (GPB7): now also J25.5 (Pin_5)
- no-connect marks 12 -> 5
Other:
- note added: "LORA COMMS"
- note added: "TODO: napraw programowanie ESPa"
- moved on the sheet: C43, C44, C49, C50, C51, C52, D8, IC2, JP10, JP6, JP7, JP8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

Commit message: WIP CMDB-Adv
Parts:
- J25: footprint (none) -> Connector_PinSocket_2.00mm:PinSocket_2x06_P2.00mm_Vertical
- R22: value 33R -> 22R; footprint Resistor_SMD:R_0805_2012Metric_Pad1.20x1.40mm_HandSolder -> Resistor_SMD:R_0402_1005Metric_Pad0.72x0.64mm_HandSolder
- R52, R53, R54, R55, R56, R57: footprint Resistor_SMD:R_0805_2012Metric_Pad1.20x1.40mm_HandSolder -> Resistor_SMD:R_0402_1005Metric_Pad0.72x0.64mm_HandSolder
Other:
- note removed: "TODO: Platform Controller IO TODO: Killswitch!!!"
- note removed: "TODO: napraw programowanie ESPa"
- moved on the sheet: C49, C50, C51, C52
