File: pcb_CMDB_Adv/ethconn.kicad_sch (KiCad schematic)
At the start: 18 parts, among them J10 ETH1, J18 ETH2

Commit message: CMDB_Adv WIP
Parts:
- added R5, R6: 0R, symbol Device:R_Small
- D12, D17: footprint (none) -> LED_SMD:LED_0603_1608Metric_Pad1.05x0.95mm_HandSolder
- R27, R35, R36, R37, R42, R43: footprint (none) -> Resistor_SMD:R_0805_2012Metric_Pad1.20x1.40mm_HandSolder
- TVS2, TVS3, TVS4, TVS5: value (none) -> TPD4E1B06
Connections:
- net 3V3 is gone; now on net +3V3: R27.2, R35.2, R36.2, R37.2
- net GND: now also R5.2, R6.2; no longer J10.SH, J18.SH
- new net: J18.SH, R6.1
- new net: J10.SH, R5.1

Commit message: WIP CMDB-Adv
Parts:
- R5, R6: footprint (none) -> Resistor_SMD:R_0805_2012Metric_Pad1.20x1.40mm_HandSolder
Changed lines of the file:
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@@
 			)
 		)
-		(property "Footprint" ""
+		(property "Footprint" "Resistor_SMD:R_0805_2012Metric_Pad1.20x1.40mm_HandSolder"
 			(at 212.09 124.46 0)
 			(hide yes)
@@
 			)
 		)
-		(property "Footprint" ""
+		(property "Footprint" "Resistor_SMD:R_0805_2012Metric_Pad1.20x1.40mm_HandSolder"
 			(at 212.09 68.58 0)
 			(hide yes)
