File: pcb_CMDB_Adv/psu.kicad_sch (KiCad schematic)
At the start: 37 parts, among them U4 AP3441SHE-7B

Commit message: CMDB-Adv PCB WIP
Parts:
- removed BT1: ML1220, symbol Device:Battery_Cell
- removed D3: NSVRB751V40T1G, Diode_SMD:D_SOD-323_HandSoldering, symbol Device:D_Schottky
- removed R6: 1K, Resistor_SMD:R_0805_2012Metric_Pad1.20x1.40mm_HandSolder, symbol Device:R
- removed TP14: +3V3SB, symbol Connector:TestPoint
- added TP19: +VIN, symbol Connector:TestPoint
- C11, C12, C13, C14, C5, C6: Distributor TME -> (none); Part Description 10uF 10% 10V Ceramic Capacitor X7R -> (none)
- C7: Distributor TME -> (none); Part Description 0.1uF 10% 16V Ceramic Capacitor X7R -> (none)
- C9: Distributor TME -> (none)
- L1: Part Description Inductor, SMT, 2520, 2u2, IRMS=7A, ISAT=8A, DCR=0.032R -> (none)
- R2: Part Description Resistor 100K M1005 1% 63mW -> (none)
- R3: Part Description Resistor 10K M1005 1% 63mW -> (none)
- R4: Part Description Resistor 2.2K M1005 1% 63mW -> (none)
- TP11, TP12, TP15, TP16, TP17, TP18, TP2, TP3, TP9: Manufacturer (none) -> -; Part No. (none) -> -
- U4: Part Description 3A DC-DC converter -> (none)
Connections:
- new net +VIN: TP19.1
Other:
- note added: "+3V3RPi"
- note added: "+3V3STB"
- note added: "+5VPB"
- note added: "+5VPB Platform Bus 5V1 - 5A (RPi) > +3V3PB1 Platform Bus 3V3 - 2.5A (PCIe) +VIMM Interm. bus 3V8 - 1.2A > +3V3PB2 Platform Bus 3V3 - 800mA (ESP32, Switch) > +3V3PB3 Platform Bus 3V3 - 300mA (LoRa) > +1V2PB Platform Bus 1V2 - 100mA (Switch) +5VEXT1 External Bus 5V1 - 4A +5VEXT2 External Bus 5V - 1.2A +3V3RPi RPi provided Bus 3V3 - 600mA +3V3STB Standby 3V3 for RTC - direct connector to RPi"
- note added: "RPi"
- note added: "TODO: - przetwornice - power or-ing - bezpieczniki - pomiar prądu - gniazda - Bulk power capacitors"
- note removed: "+3V3SB"
- note removed: "+3VSB BATT"
- note removed: "+5VPB Platform Bus 5V1 - 5A (RPi) > +3V3PB1 Platform Bus 3V3 - 2.5A (PCIe) +VIMM Interm. bus 3V8 - 1.2A > +3V3PB2 Platform Bus 3V3 - 800mA (ESP32, Switch) > +3V3PB3 Platform Bus 3V3 - 300mA (LoRa) > +1V2PB Platform Bus 1V2 - 100mA (Switch) +5VEXT1 External Bus 5V1 - 4A +5VEXT2 External Bus 5V - 1.2A +3V3RPi RPi provided Bus 3V3 - 600mA +3V3SB Standby Bus 3V3 - ~0.1mA (RPi RTC)"
- note removed: "+5VPB1"
- note removed: "TODO: - przetwornice - power or-ing - bezpieczniki - pomiar prądu - gniazda"
- note removed: "standby LDO"
- moved on the sheet: TP15

Commit message: CMDB_Adv WIP
Parts:
- removed C11, C12, C13, C14, C5, C6: 10u, Capacitor_SMD:C_0805_2012Metric_Pad1.18x1.45mm_HandSolder, symbol Device:C
- removed C17: BULK_VIN_CAP, symbol Device:C_Polarized
- removed C7: 100n, Capacitor_SMD:C_0805_2012Metric_Pad1.18x1.45mm_HandSolder, symbol Device:C
- removed C9: 4.7nF, Capacitor_SMD:C_0805_2012Metric_Pad1.18x1.45mm_HandSolder, symbol Device:C
- removed D2: +3V3PB1, Diode_SMD:D_0805_2012Metric_Pad1.15x1.40mm_HandSolder, symbol Device:D_Small_Filled
- removed L1: 2.2uH, CMDB_Adv:L_Bourns_SRP5030CC, symbol Device:L
- removed R2: 100K, Resistor_SMD:R_0805_2012Metric_Pad1.20x1.40mm_HandSolder, symbol Device:R
- removed R3: 10K, Resistor_SMD:R_0805_2012Metric_Pad1.20x1.40mm_HandSolder, symbol Device:R
- removed R4: 2.2K, Resistor_SMD:R_0805_2012Metric_Pad1.20x1.40mm_HandSolder, symbol Device:R
- removed R5: 1K, Resistor_SMD:R_0805_2012Metric_Pad1.20x1.40mm_HandSolder, symbol Device:R_Small
- removed U4: AP3441SHE-7B, Package_DFN_QFN:DFN-8-1EP_2x2mm_P0.5mm_EP1.05x1.75mm, symbol CM5IO:AP3441SHE-7B
- added C54, C55, C57, C59, C63: 100nF, Capacitor_SMD:C_0402_1005Metric_Pad0.74x0.62mm_HandSolder, symbol Device:C_Small
- added C56, C60: 47uF, symbol Device:C_Polarized
- added C65, C66, C67, C68, C69, C70: 10uF, Capacitor_SMD:C_1206_3216Metric_Pad1.33x1.80mm_HandSolder, symbol Device:C_Small
- added D2, D9: SS34, Diode_SMD:D_SMA_Handsoldering, symbol Device:D_Schottky
- added JP12: +3V3PB2 DIS, Jumper:SolderJumper-3_P1.3mm_Bridged12_RoundedPad1.0x1.5mm, symbol Jumper:SolderJumper_3_Bridged12
- added JP13: +3V3PB3 DIS, Jumper:SolderJumper-3_P1.3mm_Bridged12_RoundedPad1.0x1.5mm, symbol Jumper:SolderJumper_3_Bridged12
- added JP14: +1V2PB DIS, Jumper:SolderJumper-3_P1.3mm_Bridged12_RoundedPad1.0x1.5mm, symbol Jumper:SolderJumper_3_Bridged12
- added Q1, Q2: AON7534, Package_DFN_QFN:DFN-8-1EP_3x3mm_P0.65mm_EP1.6x2.56mm_ThermalVias, symbol Simulation_SPICE:NMOS
- added R12, R3: 3K57, symbol Device:R_Small
- added R23, R4: 1K15, symbol Device:R_Small
- added R40: 5K9, symbol Device:R_Small
- added R45: 11K8, symbol Device:R_Small
- added R48, R49, R50, R51: 10K, symbol Device:R_Small
- added U2, U3: LM74700, Package_TO_SOT_SMD:SOT-23-6, symbol Power_Management:LM74700
- added U4, U8, U9: TPS7A91, Package_DFN_QFN:Texas_S-PDSO-N10_EP1.2x2mm, symbol Regulator_Linear:TPS7A91
- TP11, TP12, TP15, TP16, TP17, TP18, TP19, TP2, TP3, TP9: footprint (none) -> TestPoint:TestPoint_Pad_1.5x1.5mm
Connections:
- net +1V2PB: now also C66.1, R40.1, U9.1 (OUT), U9.2 (OUT)
- net +3V3PB1_EN: now also R50.1
- net +3V3PB2: now also C67.1, R3.1, R48.2, R49.2, R50.2, R51.2, U4.1 (OUT), U4.2 (OUT)
- net +3V3PB3: now also C68.1, R12.1, U8.1 (OUT), U8.2 (OUT)
- net +5VEXT1_EN: now also R49.1
- net +5VEXT2_EN: now also R48.1
- net +5VPB: now also C56.1, Q1.1 (D), Q2.1 (D), U2.4 (CATHODE), U3.4 (CATHODE)
- net +5VPB_EN: now also R51.1
- net +VBUS_USBC: now also C55.2, D2.2 (A), Q2.3 (S), U3.3 (EN), U3.6 (ANODE)
- net +VIMM: now also C60.1, C65.1, C69.1, C70.1, D2.1 (K), D9.1 (K), JP12.1 (A), JP13.1 (A), JP14.1 (A), U4.10 (IN), U4.9 (IN), U8.10 (IN), U8.9 (IN), U9.10 (IN), U9.9 (IN)
- net GND: now also C56.2, C57.1, C59.1, C60.2, C63.1, C65.2, C66.2, C67.2, C68.2, C69.2, C70.2, JP12.3 (B), JP13.3 (B), JP14.3 (B), R23.2, R4.2, R45.2, U2.2 (GND), U3.2 (GND), U4.11 (GND), U4.4 (GND), U4.6 (SS_CTRL), U8.11 (GND), U8.4 (GND), U8.6 (SS_CTRL), U9.11 (GND), U9.4 (GND), U9.6 (SS_CTRL)
- new net: R12.2, R23.1, U8.3 (FB)
- new net: R40.2, R45.1, U9.3 (FB)
- new net: C57.2, U4.8 (NR/SS)
- new net: R3.2, R4.1, U4.3 (FB)
- new net: C63.2, U9.8 (NR/SS)
- new net: C55.1, U3.1 (VCAP)
- new net: Q2.2 (G), U3.5 (GATE)
- new net: JP12.2 (C), U4.7 (EN)
- new net: C59.2, U8.8 (NR/SS)
- new net: JP14.2 (C), U9.7 (EN)
- new net: C54.1, U2.1 (VCAP)
- new net: JP13.2 (C), U8.7 (EN)
- new net: Q1.2 (G), U2.5 (GATE)
- new net PSU Converters/+5VPB: C54.2, Q1.3 (S), U2.3 (EN), U2.6 (ANODE)
- new net PSU Converters/+VIMM: D9.2 (A)
- no-connect marks 1 -> 3
Other:
- added sheet PSU Converters (psu_converters.kicad_sch)
- note added: "+5VPB_EN has no effect when powering device from USB"
- note added: "+VBUS_USBC"
- note added: "+VIN"
- note added: "+VIN can be 3s-8s, charged or dying. I.e. 9V-33.6V"
- note added: "DC-DC"
- note added: "IF VBUS_USB is present, and VIN is not, VIMM should be generated from VBUS_USB. In such case, 5VPB should be fed directly from VBUS_USB voltage."
- note added: "PMIC/multiple DC-DC converters"
- note added: "TODO: - Bulk power capacitors - Bezpieczniki (Poly? eFuse?) - ESD na VIN oraz VBUS - Power Valid (Zielona dioda, I guess)"
- note added: "VIMM converter should output a little higher voltage to compensate for shottky diode drop (~4.3V ?)"
- note added: "Voltage OR-ing circuits"
- note removed: "AP3441"
- note removed: "PMIC/multiple converters"
- note removed: "PSU_MAX_CURRENT=5000 must be set in rpi-eeprom-config to allow full power at USB ports"
- note removed: "TODO: - przetwornice - power or-ing - bezpieczniki - pomiar prądu - gniazda - Bulk power capacitors"
- note removed: "VBUS_USB"
- note removed: "VIN"
- moved on the sheet: D10, R26, TP15, TP16, TP18, TP19, TP2, TP9

Commit message: WIP
Parts:
- removed TP2: +5VPB, TestPoint:TestPoint_Pad_1.5x1.5mm, symbol Connector:TestPoint
- added D11: +5VPB, Diode_SMD:D_0805_2012Metric_Pad1.15x1.40mm_HandSolder, symbol Device:D_Small_Filled
- added J1: RFShield_OnePiece, symbol Device:RFShield_OnePiece
- added R58: 1K, Resistor_SMD:R_0805_2012Metric_Pad1.20x1.40mm_HandSolder, symbol Device:R_Small
- added TP4: +5VPB, TestPoint:TestPoint_Pad_1.5x1.5mm, symbol Connector:TestPoint
- D10: value +5VPB -> PWR_VALID
Connections:
- net +5VPB: now also D11.2 (A), TP4.1; no longer D10.2 (A)
- net GND: now also J1.1 (Shield), R58.2
- new net: D11.1 (K), R58.1
- new net POWER_VALID: D10.2 (A)
Other:
- note added: "+5VPB Platform Bus 5V1 - 5A (RPi) > +3V3PB1 Platform Bus 3V3 - 2.5A (PCIe) +VIMM Interm. bus 3V8 - 1.2A > +3V3PB2 Platform Bus 3V3 - 800mA (ESP32, Switch) > +3V3PB3 Platform Bus 3V3 - 300mA (LoRa) > +1V2PB Platform Bus 1V2 - 100mA (Switch) +5VEXT1 External Bus 5V1 - 4A min. +5VEXT2 External Bus 5V1 - 4A min. +3V3RPi RPi provided Bus 3V3 - 600mA +3V3STB Standby 3V3 for RTC - direct connector to RPi"
- note added: "+VIN can be 3s-6s, charged or dying. I.e. 9V-25.2V"
- note added: "PSU should be contained under this shield"
- note added: "TODO: - Bezpieczniki (Poly? eFuse?) - TVS na VIN oraz VBUS"
- note removed: "+5VPB Platform Bus 5V1 - 5A (RPi) > +3V3PB1 Platform Bus 3V3 - 2.5A (PCIe) +VIMM Interm. bus 3V8 - 1.2A > +3V3PB2 Platform Bus 3V3 - 800mA (ESP32, Switch) > +3V3PB3 Platform Bus 3V3 - 300mA (LoRa) > +1V2PB Platform Bus 1V2 - 100mA (Switch) +5VEXT1 External Bus 5V1 - 4A +5VEXT2 External Bus 5V - 1.2A +3V3RPi RPi provided Bus 3V3 - 600mA +3V3STB Standby 3V3 for RTC - direct connector to RPi"
- note removed: "+VIN can be 3s-8s, charged or dying. I.e. 9V-33.6V"
- note removed: "TODO: - Bulk power capacitors - Bezpieczniki (Poly? eFuse?) - ESD na VIN oraz VBUS - Power Valid (Zielona dioda, I guess)"
- moved on the sheet: C55, D10, D13, D14, D16, R26, R29, R30, R32, TP11, TP12, TP15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

Commit message: WIP CMDB-Adv
Parts:
- R12, R23, R3, R4, R40, R45, R48, R49, R50, R51: footprint (none) -> Resistor_SMD:R_0805_2012Metric_Pad1.20x1.40mm_HandSolder
Changed lines of the file:
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@@
 			)
 		)
-		(property "Footprint" ""
+		(property "Footprint" "Resistor_SMD:R_0805_2012Metric_Pad1.20x1.40mm_HandSolder"
 			(at 264.16 78.74 0)
 			(hide yes)
@@
 			)
 		)
-		(property "Footprint" ""
+		(property "Footprint" "Resistor_SMD:R_0805_2012Metric_Pad1.20x1.40mm_HandSolder"
 			(at 49.53 67.31 0)
 			(hide yes)
@@
 			)
 		)
-		(property "Footprint" ""
+		(property "Footprint" "Resistor_SMD:R_0805_2012Metric_Pad1.20x1.40mm_HandSolder"
 			(at 68.58 67.31 0)
 			(hide yes)
@@
 			)
 		)
-		(property "Footprint" ""
+		(property "Footprint" "Resistor_SMD:R_0805_2012Metric_Pad1.20x1.40mm_HandSolder"
 			(at 264.16 113.03 0)
 			(hide yes)
@@
 			)
 		)
-		(property "Footprint" ""
+		(property "Footprint" "Resistor_SMD:R_0805_2012Metric_Pad1.20x1.40mm_HandSolder"
 			(at 264.16 45.72 0)
 			(hide yes)
@@
 			)
 		)
-		(property "Footprint" ""
+		(property "Footprint" "Resistor_SMD:R_0805_2012Metric_Pad1.20x1.40mm_HandSolder"
 			(at 264.16 40.64 0)
 			(hide yes)
@@
 			)
 		)
-		(property "Footprint" ""
+		(property "Footprint" "Resistor_SMD:R_0805_2012Metric_Pad1.20x1.40mm_HandSolder"
 			(at 264.16 107.95 0)
 			(hide yes)
@@
 			)
 		)
-		(property "Footprint" ""
+		(property "Footprint" "Resistor_SMD:R_0805_2012Metric_Pad1.20x1.40mm_HandSolder"
 			(at 55.88 67.31 0)
 			(hide yes)
@@
 			)
 		)
-		(property "Footprint" ""
+		(property "Footprint" "Resistor_SMD:R_0805_2012Metric_Pad1.20x1.40mm_HandSolder"
 			(at 62.23 67.31 0)
 			(hide yes)
@@
 			)
 		)
-		(property "Footprint" ""
+		(property "Footprint" "Resistor_SMD:R_0805_2012Metric_Pad1.20x1.40mm_HandSolder"
 			(at 264.16 73.66 0)
 			(hide yes)
