File: pcb_CMDB_Adv/psu_converters.kicad_sch (KiCad schematic)
At the start: 9 parts, among them U10 INA3221, U11 INA3221

Commit message: WIP
Parts:
- added J24: AUX_PWR, symbol Connector_Generic:Conn_02x04_Counter_Clockwise
- added TP13: PWR_VALID1, TestPoint:TestPoint_Pad_1.5x1.5mm, symbol Connector:TestPoint
- added TP5: PWR_VALID0, TestPoint:TestPoint_Pad_1.5x1.5mm, symbol Connector:TestPoint
Connections:
- net +5VPB: now also J24.1 (Pin_1)
- net +VIMM: now also J24.8 (Pin_8)
- net +VIN: now also J24.2 (Pin_2), J24.3 (Pin_3), J24.4 (Pin_4)
- net GND: now also J24.5 (Pin_5), J24.6 (Pin_6), J24.7 (Pin_7)
- net POWER_VALID0: now also TP5.1
- net POWER_VALID1: now also TP13.1
Other:
- note added: "TODO: - przetwornice - pomiar napięcia/prądu (INA3221) +VBUS_USBC +VIN +5VPB&+3V3PB1 +5VIMM +5VEXT1 +5VEXT2 - assign POWER_VALID = (POWER_VALID0 && POWER_VALID1) Nie ma VIMM_EN - zawsze jest włączone. STAN WYSOKI NA PINACH EN TO +3V3!"
- note removed: "TODO: - przetwornice - pomiar napięcia/prądu (INA3221) +VBUS_USBC +VIN +5VPB&+3V3PB1 +5VIMM +5VEXT1 +5VEXT2 Nie ma VIMM_EN - zawsze jest włączone. STAN WYSOKI NA PINACH EN TO +3V3!"

Commit message: WIP CMDB-Adv
Parts:
- added J27: AUX_PWR_OUT2, Connector_PinSocket_2.00mm:PinSocket_2x04_P2.00mm_Vertical, symbol Connector_Generic:Conn_02x04_Counter_Clockwise
- J24: value AUX_PWR -> AUX_PWR_OUT1; footprint (none) -> Connector_PinSocket_2.00mm:PinSocket_2x04_P2.00mm_Vertical
Connections:
- net +5VPB: now also J27.5 (Pin_5), J27.6 (Pin_6); no longer J24.1 (Pin_1)
- net +VIMM: now also J27.7 (Pin_7), J27.8 (Pin_8); no longer J24.8 (Pin_8)
- net +VIN: now also J24.5 (Pin_5), J24.6 (Pin_6), J24.7 (Pin_7), J24.8 (Pin_8); no longer J24.2 (Pin_2), J24.3 (Pin_3)
- net GND: now also J24.1 (Pin_1), J24.2 (Pin_2), J24.3 (Pin_3), J27.1 (Pin_1), J27.2 (Pin_2), J27.3 (Pin_3), J27.4 (Pin_4); no longer J24.5 (Pin_5), J24.6 (Pin_6), J24.7 (Pin_7)
